File: base/Schematics and Boards/cs_v2.sch (EAGLE design)
At the start: 73 parts, among them J1 J-MICROSD-DM3AT-SF-PEJM5, J3 J-JTAG-CORTEX-NEEDLE6, Q1 DMG3415UFY4Q-7, Q2 FK3303010L, Q3 FK3303010L, Q4 FK3303010L, U1 ATSAMD51, U2 MAX77827BEWC+T, U202 COULOMB-MAX17262, U206 LOADSWITCH-MIC94162, U3 PD3S140-7, Y1 16M, Y2 ABS07-32.768KHZ-9-T

Commit message: Processor wired up
Parts:
- added C22: 0.1u, Capacitors:C-0402
- added C23: 1u, Capacitors:C-0603
- added J_DTR1: HIROSE-DF40_80-PIN_CONNECTORS, Connectors:HIROSE-DF40_80-PIN_CONNECTORS
- added R10, R11: 4.7k, Resistors:R-0402
- added R_SENSE_TEMP: 10, Resistors:R-0603
- added U4: SENSOR-SI7006, Sensors:SENSOR-SI7006
- added U5: LOADSWITCH-MIC94162, Switches:LOADSWITCH-MIC94162
- J2: device Connectors:J-JST2-SMT_RA-SH -> Connectors:J-JST2-SMT-RA
- R_SENSE_DTR: value 0.5 -> 0.51; PART_NO ERJ-3RQFR51V -> ERJ-3BQFR51V
Connections:
- net DTR_BUS3_SERCOM3_P2 renamed DBG_USB_D-
- net DTR_BUS3_SERCOM3_P3 renamed DBG_USB_D+
- removed net DBG_SWO: J3.SWO, U1.PB30
- removed net DTR_BUS3_SERCOM3_P0: U1.PA22
- removed net DTR_BUS3_SERCOM3_P1: U1.PA23
- new net +3V3_TEMP: C22.1, U4.V, U5.VOUT
- new net +3V3_TEMP_SENSE: C23.1, R_SENSE_TEMP.2, U5.VIN
- new net DBG_GPIO0: U1.PC16
- new net DBG_GPIO1: U1.PC17
- new net DBG_GPIO2: U1.PC18
- new net DBG_GPIO3: U1.PC19
- new net DBG_TRACE_CLK: U1.PC27
- new net DBG_TRACE_D0: U1.PC28
- new net DBG_TRACE_D1: U1.PC26
- new net DBG_TRACE_D2: U1.PC25
- new net DBG_TRACE_D3: U1.PC24
- new net DBG_TRACE_SWO: U1.PB30
- new net DTR_BUS0_AIN1: U1.PA3
- new net DTR_BUS0_GPIO0: U1.PB12
- new net DTR_BUS0_GPIO1: U1.PB13
- new net DTR_BUS1_AIN1: U1.PA5
- new net DTR_BUS1_GPIO0: U1.PB14
- new net DTR_BUS1_GPIO1: U1.PB15
- new net DTR_BUS2_AIN1: U1.PC3
- new net DTR_BUS2_GPIO0: U1.PB16
- new net DTR_BUS2_GPIO1: U1.PB17
- new net DTR_BUS3_AIN1: U1.PB5
- new net DTR_BUS3_GPIO0: U1.PA6
- new net DTR_BUS3_GPIO1: U1.PA7
- new net DTR_BUS3_SERCOM7_P0: U1.PD8
- new net DTR_BUS3_SERCOM7_P1: U1.PD9
- new net DTR_BUS3_SERCOM7_P2: U1.PD10
- new net DTR_BUS3_SERCOM7_P3: U1.PD11
- new net DTR_DETECT: U1.PC31
- new net EN_TEMP: U5.ENABLE
- net +3V3: now also L2.2, R_SENSE_TEMP.1
- net +3V3_PROC: now also R10.2, R11.2; no longer L2.2
- net DTR_BUS0_AIN0: now also U1.PA2; no longer U1.PC0
- net DTR_BUS0_SERCOM0_P0: now also U1.PA8; no longer U1.PC17
- net DTR_BUS0_SERCOM0_P1: now also U1.PA9; no longer U1.PC16
- net DTR_BUS0_SERCOM0_P2: now also U1.PA10; no longer U1.PC18
- net DTR_BUS0_SERCOM0_P3: now also U1.PA11; no longer U1.PC19
- net DTR_BUS1_AIN0: now also U1.PA4; no longer U1.PC1
- net DTR_BUS2_SERCOM2_P0: now also U1.PA12; no longer U1.PB26
- net DTR_BUS2_SERCOM2_P1: now also U1.PA13; no longer U1.PB27
- net DTR_BUS2_SERCOM2_P2: now also U1.PA14; no longer U1.PB28
- net DTR_BUS2_SERCOM2_P3: now also U1.PA15; no longer U1.PB29
- net DTR_BUS3_AIN0: now also U1.PB4; no longer U1.PC3
- net DTR_MASTER_I2C_SCL: now also R10.1, U1.PA23, U4.SCL; no longer U1.PB3
- net DTR_MASTER_I2C_SDA: now also R11.1, U1.PA22, U4.SDA; no longer U1.PB2
- net GND: now also C22.2, C23.2, J2.1, U4.GND, U5.GND; no longer J2.2
- net LED_B: now also U1.PB28
- net LED_G: now also U1.PB27
- net LED_R: now also U1.PB26
- net N$7: now also J2.2; no longer J2.1
- net SD_CD: now also U1.PD20; no longer U1.PA6
- net SD_CLK: now also U1.PA21; no longer U1.PB11
- net SD_CMD: now also U1.PA20; no longer U1.PA8
- net SD_D0: now also U1.PB18; no longer U1.PA9
- net SD_D1: now also U1.PB19; no longer U1.PA10
- net SD_D2: now also U1.PB20; no longer U1.PA11
- net SD_D3: now also U1.PB21; no longer U1.PB10
- net XIN: now also U1.PB22; no longer U1.PA14
- net XOUT: now also U1.PB23; no longer U1.PA15
Other:
- note added: "Debugger Tag Connect"
- note added: "I2C Pull-ups"
- note added: "Provide info on board health (humitidy/temp) and info to help with crystal frequency offset resulting from temperature"
- note added: "SD Card"
- note added: "Says to connect AGND to PGND on PCB low impedance plane, away from any critical loops"
- note added: "Temperature Sensor"
- note removed: "Debugger Connect"
- note removed: "Route analog signals through this resistor. The resistor is big and fat for this purpose!"
- note removed: "Sense resistor values are suggetions. These values may need to be updated. They should, for max current draw, have no more than 100 mV drop on 3.3V output."
- note removed: "Using SH type connector (1mm pitch), as opposed to PH type (2mm pitch). Height chopped in half, but carries less current (1A rating) and is more prone to rip off. Unlikely to find many batteries with this connector by default."
- moved on the sheet: J2

Commit message: Wire up connectors. Schematic complete, awaiting review
Parts:
- removed J_DTR1: HIROSE-DF40_80-PIN_CONNECTORS, Connectors:HIROSE-DF40_80-PIN_CONNECTORS
- added J_DBG: HIROSE-DF40_30-PIN_CONNECTORS-RECEPTACLE, Connectors:HIROSE-DF40_30-PIN_CONNECTORS-RECEPTACLE
- J_DTR: value HIROSE-DF40_80-PIN_CONNECTORS -> HIROSE-DF40_44-PIN_CONNECTORS-RECEPTACLE; device Connectors:HIROSE-DF40_80-PIN_CONNECTORS -> Connectors:HIROSE-DF40_44-PIN_CONNECTORS-RECEPTACLE
Connections:
- new net N$21: J_DBG.1, J_DBG.3, J_DBG.5
- net +3V3: now also J_DBG.12
- net +3V3_DTR: now also J_DBG.16, J_DTR.2, J_DTR.4, J_DTR.6
- net +3V3_PROC: now also J_DBG.14
- net +3V3_SD_SENSE: now also J_DBG.18
- net +3V3_TEMP_SENSE: now also J_DBG.20
- net +3V7_BATT: now also J_DBG.10, J_DBG.6, J_DBG.8
- net DBG_GPIO0: now also J_DBG.7
- net DBG_GPIO1: now also J_DBG.9
- net DBG_GPIO2: now also J_DBG.11
- net DBG_GPIO3: now also J_DBG.13
- net DBG_SERIAL_RX: now also J_DBG.17
- net DBG_SERIAL_TX: now also J_DBG.15
- net DBG_SWCLK: now also J_DBG.19
- net DBG_SWDIO: now also J_DBG.21
- net DBG_TRACE_CLK: now also J_DBG.26
- net DBG_TRACE_D0: now also J_DBG.23
- net DBG_TRACE_D1: now also J_DBG.25
- net DBG_TRACE_D2: now also J_DBG.27
- net DBG_TRACE_D3: now also J_DBG.29
- net DBG_TRACE_SWO: now also J_DBG.28
- net DBG_USB_D+: now also J_DBG.24
- net DBG_USB_D-: now also J_DBG.22
- net DTR_BUS0_AIN0: now also J_DTR.8
- net DTR_BUS0_AIN1: now also J_DTR.16
- net DTR_BUS0_GPIO0: now also J_DTR.24
- net DTR_BUS0_GPIO1: now also J_DTR.32
- net DTR_BUS0_SERCOM0_P0: now also J_DTR.7
- net DTR_BUS0_SERCOM0_P1: now also J_DTR.15
- net DTR_BUS0_SERCOM0_P2: now also J_DTR.23
- net DTR_BUS0_SERCOM0_P3: now also J_DTR.31
- net DTR_BUS1_AIN0: now also J_DTR.10
- net DTR_BUS1_AIN1: now also J_DTR.18
- net DTR_BUS1_GPIO0: now also J_DTR.26
- net DTR_BUS1_GPIO1: now also J_DTR.34
- net DTR_BUS1_SERCOM1_P0: now also J_DTR.9
- net DTR_BUS1_SERCOM1_P1: now also J_DTR.17
- net DTR_BUS1_SERCOM1_P2: now also J_DTR.25
- net DTR_BUS1_SERCOM1_P3: now also J_DTR.33
- net DTR_BUS2_AIN0: now also J_DTR.12
- net DTR_BUS2_AIN1: now also J_DTR.20
- net DTR_BUS2_GPIO0: now also J_DTR.28
- net DTR_BUS2_GPIO1: now also J_DTR.36
- net DTR_BUS2_SERCOM2_P0: now also J_DTR.11
- net DTR_BUS2_SERCOM2_P1: now also J_DTR.19
- net DTR_BUS2_SERCOM2_P2: now also J_DTR.27
- net DTR_BUS2_SERCOM2_P3: now also J_DTR.35
- net DTR_BUS3_AIN0: now also J_DTR.14
- net DTR_BUS3_AIN1: now also J_DTR.22
- net DTR_BUS3_GPIO0: now also J_DTR.30
- net DTR_BUS3_GPIO1: now also J_DTR.38
- net DTR_BUS3_SERCOM7_P0: now also J_DTR.13
- net DTR_BUS3_SERCOM7_P1: now also J_DTR.21
- net DTR_BUS3_SERCOM7_P2: now also J_DTR.29
- net DTR_BUS3_SERCOM7_P3: now also J_DTR.37
- net DTR_DETECT: now also J_DTR.39
- net DTR_MASTER_I2C_SCL: now also J_DTR.40
- net DTR_MASTER_I2C_SDA: now also J_DTR.42
- net GND: now also J_DTR.1, J_DTR.3, J_DTR.5
- net NRESET: now also J_DBG.30
- net VDD_DBG: now also J_DBG.2, J_DBG.4
Other:
- note added: "External Connectors"
- note added: "Idea: put similar pins (rather than SERCOM buses) right next to each other to make passthrough easier for dtr boards"
- note removed: "Pinout Headers"
- moved on the sheet: C20, C21, C22, C23, JP3, JP4, R_SENSE_DTR, R_SENSE_PROC, R_SENSE_SD, R_SENSE_TEMP, U206, U5

Commit message: Minor changes based on schematic review
Ready to generate board and work on layout. Should be careful to ensure that 3V3 is indeed isolated from the other 3V3 lines -- there is some weirdness related to 3v3 supply symbols and connecting differently named nets to said symbols.
Parts:
- removed R3: 0, Resistors:R-2010
- JP1, JP2, JP3, JP4: value JUMPER-SMT_2_NC_PASTE_SILK -> JUMPER-SMT_2_NC_PASTE_NO-SILK; device SparkFun-Jumpers:JUMPER-SMT_2_NC_PASTE_SILK -> Connectors:JUMPER-SMT_2_NC_PASTE_NO-SILK
- R5: value 150 -> 1k; PART_NO ERJ-2GEJ151X -> ERA-2AED102X; TOL (none) -> 0.5%
- R6, R7: value 30 -> 590; PART_NO ERJ-2RKF30R0X -> ERJ-2RKF5900X; TOL (none) -> 1%
- S2: PART_NO (none) -> CUS-12TB
- U206, U5: value LOADSWITCH-MIC94162 -> LOADSWITCH-MIC94164; device Switches:LOADSWITCH-MIC94162 -> Switches:LOADSWITCH-MIC94164
Connections:
- removed net AGND: C_REG_BIAS.2, R3.1, U2.AGND
- net +3V3: no longer L2.2
- net +3V3_PROC: now also L2.2
- net GND: now also C_REG_BIAS.2, U2.AGND; no longer R3.2
Other:
- note added: "Aim for 1 mA output for each LED. Green (1) and Blue(3) have forward biases near 3V, so no resistor needed. Red (2) has forward bias 1.8V. Outputs of this should be tied to GND by processor to turn an LED on."
- note removed: "Aim for 10 mA output for each LED. Green (1) and Blue(3) have forward biases near 3V, so no resistor needed. Red (2) has forward bias 1.8V. Outputs of this should be tied to GND by processor to turn an LED on."
- note removed: "Ground Connection"

Commit message: Move CC after power selection. Add SPI flash over SD. Swap PowSel diode
Parts:
- removed C21: 1u, Capacitors:C-0603
- removed C_REG_BIAS: 1u, Capacitors:C-0402
- removed C_REG_IN: 10u, Capacitors:C-0603
- removed C_REG_OUT: 22u, Capacitors:C-0805
- removed J1: J-MICROSD-DM3AT-SF-PEJM5, Connectors:J-MICROSD-DM3AT-SF-PEJM5
- removed J2: (no value), Connectors:J-JST2-SMT-RA
- removed JP2: JUMPER-SMT_2_NC_PASTE_NO-SILK, Connectors:JUMPER-SMT_2_NC_PASTE_NO-SILK
- removed L3: 1u, Inductors:L1008
- removed Q1: DMG3415UFY4Q-7, Switches:DMG3415UFY4Q-7
- removed R4: 100k, Resistors:R-0402
- removed R_SDCMD: 10K, Resistors:R-0402
- removed R_SDDAT0, R_SDDAT1, R_SDDAT2, R_SDDAT3: 100K, Resistors:R-0402
- removed R_SD_DET1: 510k, Resistors:R-0402
- removed S1: MOMENTARY-SWITCH-SPST-SMD-4.6X2.8MM, SparkFun-Switches:MOMENTARY-SWITCH-SPST-SMD-4.6X2.8MM
- removed S2: (no value), Switches:SLIDESWITCH-SPDT-SMD-RIGHT-ANGLE
- removed TP1, TP2: PTR1TP19R, TestPoints:PTR1TP19R
- removed U2: MAX77827BEWC+T, Regulators:MAX77827BEWC+T
- removed U3: PD3S140-7, Diodes:PD3S140-7
- removed U5: LOADSWITCH-MIC94164, Switches:LOADSWITCH-MIC94164
- added C201: 100n, Capacitors:C-0402
- added C203: 470n, Capacitors:C-0402
- added C204: 1u, Capacitors:C-0402
- added C205: 22u, Capacitors:C-0805
- added J201: (no value), Connectors:J-JST2-SMT-RA
- added JP_VDBG: JUMPER-SMT_2_NC_PASTE_NO-SILK, Connectors:JUMPER-SMT_2_NC_PASTE_NO-SILK
- added L201: 1u, Inductors:L1008
- added Q204: DMG3415UFY4Q-7, Switches:DMG3415UFY4Q-7
- added R204: 10M, Resistors:R-0402
- added S101: SW_EVQ-P7L01P_SPST_RA, Switches:SW_EVQ-P7L01P_SPST_RA
- added S201: (no value), Switches:SLIDESWITCH-SPDT-SMD-RIGHT-ANGLE
- added U101: ATSAMD51, Processors:ATSAMD51
- added U201: COULOMB-MAX17262, CoulombCounters:COULOMB-MAX17262
- added U203: MAX77827BEWC+T, Regulators:MAX77827BEWC+T
- added U205: LOADSWITCH-MIC94164, Switches:LOADSWITCH-MIC94164
- C202: value 100n -> 10u; device Capacitors:C-0402 -> Capacitors:C-0603; MP CC0402KRX5R5BB104 -> (none); PART_NO (none) -> C0603C106M8PAC7867; TC (none) -> X5R; VOLTAGE (none) -> 10V
- C206: value 470n -> 1u; device Capacitors:C-0402 -> Capacitors:C-0603; MP CC0402KRX5R5BB474 -> (none); PART_NO (none) -> C0603C105K8RACTU; VOLTAGE (none) -> 10V
- TP3, TP4: value PTR1TP19R -> TPTP08R; device TestPoints:PTR1TP19R -> TestPoints:TPTP08R
- U1: value ATSAMD51 -> AT25SF641-MHB-T; device Processors:ATSAMD51 -> Storage:AT25SF641-MHB-T
- U202: value COULOMB-MAX17262 -> CUS520H3F; device CoulombCounters:COULOMB-MAX17262 -> Diodes:CUS520H3F; MP MAX17262REWL+T -> (none)
- renumbered C1 to C107, C10 to C115, C11 to C105, C12 to C108, C13 to C110, C14 to C114, C15 to C101, C16 to C116, C17 to C117, C18 to C118, C19 to C119, C2 to C103, C20 to C208, C22 to C209, C23 to C207, C3 to C102, C4 to C104, C5 to C106, C6 to C109, C7 to C111, C8 to C112, C9 to C113, D1 to D201, J3 to J101, JP1 to JP202, JP3 to JP204, JP4 to JP_PROC, J_DBG to J302, J_DTR to J301, L1 to L101, L2 to L102, Q2 to Q201, Q3 to Q202, Q4 to Q203, R1 to R101, R10 to R103, R11 to R104, R2 to R102, R5 to R203, R6 to R201, R7 to R202, R8 to R112, R9 to R106, R_SENSE_DTR to R207, R_SENSE_PROC to R206, R_SENSE_SD to R208, R_SENSE_TEMP to R205, U4 to U204, Y1 to Y101, Y2 to Y102
Connections:
- removed net +3V3_SD: C208.1, J1.VDD, R_SDCMD.2, R_SDDAT0.2, R_SDDAT1.2, R_SDDAT2.2, R_SDDAT3.2, R_SD_DET1.1, TP2.TP, U206.VOUT
- removed net +3V3_SD_SENSE: C21.1, J302.18, R208.2, U206.VIN
- removed net +3V7_BATT_IN: C202.1, S2.S, U202.BATT, U202.TH
- removed net BATT_ALERT: U202.ALRT
- removed net EN_SD: U206.ENABLE
- removed net N$7: J2.2, S2.P
- removed net N$8: S2.O
- removed net SD_CD: J1.A, R_SD_DET1.2, U1.PD20
- removed net SD_CLK: J1.CLK, U1.PA21
- removed net SD_CMD: J1.CMD, R_SDCMD.1, U1.PA20
- removed net SD_D0: J1.DAT0, R_SDDAT0.1, U1.PB18
- removed net SD_D1: J1.DAT1, R_SDDAT1.1, U1.PB19
- removed net SD_D2: J1.DAT2, R_SDDAT2.1, U1.PB20
- removed net SD_D3: J1.CD/DAT3, R_SDDAT3.1, U1.PB21
- new net +3V3_STOR: C208.1, U1.VDD, U205.VOUT
- new net +3V3_STOR_SENSE: C206.1, J302.18, R208.2, U205.VIN
- new net CC_IN: C201.1, S201.O, U201.BATT, U201.TH
- new net EN_STOR: U101.PC6, U205.ENABLE
- new net STOR_HOLD: U1.NHOLD/IO3, U101.PB7
- new net STOR_SPI5_MISO: U1.SO/IO1, U101.PB3
- new net STOR_SPI5_MOSI: U1.SI/IO0, U101.PB0
- new net STOR_SPI5_NCS: U1.NCS, U101.PB2
- new net STOR_SPI5_SCK: U1.SCK, U101.PB1
- new net STOR_WP: U1.WP/IO2, U101.PB6
- new net VDD_SW: Q204.S, S201.P, U202.N
- net +3V3: now also C205.1, U203.OUT, U203.OUTS; no longer C_REG_OUT.1, U2.OUT, U2.OUTS
- net +3V3_PROC: now also U101.VDDIO3, U101.VDDIO4, U101.VDDIO5, U101.VDDIO6, U101.VDDIO7, U101.VDDIOB1, U101.VDDIOB2; no longer U1.VDDIO3, U1.VDDIO4, U1.VDDIO5, U1.VDDIO6, U1.VDDIO7, U1.VDDIOB1, U1.VDDIOB2
- net +3V3_TEMP: now also U206.VOUT; no longer U5.VOUT
- net +3V3_TEMP_SENSE: now also U206.VIN; no longer U5.VIN
- net +3V7_BATT: now also J201.2, Q204.D; no longer Q1.D, TP1.TP, U202.SYS
- net DBG_GPIO0: now also U101.PC16; no longer U1.PC16
- net DBG_GPIO1: now also U101.PC17; no longer U1.PC17
- net DBG_GPIO2: now also U101.PC18; no longer U1.PC18
- net DBG_GPIO3: now also U101.PC19; no longer U1.PC19
- net DBG_SERIAL_RX: now also U101.PB9; no longer U1.PB9
- net DBG_SERIAL_TX: now also U101.PB8; no longer U1.PB8
- net DBG_SWCLK: now also U101.PA30; no longer U1.PA30
- net DBG_SWDIO: now also U101.PA31; no longer U1.PA31
- net DBG_TRACE_CLK: now also U101.PC27; no longer U1.PC27
- net DBG_TRACE_D0: now also U101.PC28; no longer U1.PC28
- net DBG_TRACE_D1: now also U101.PC26; no longer U1.PC26
- net DBG_TRACE_D2: now also U101.PC25; no longer U1.PC25
- net DBG_TRACE_D3: now also U101.PC24; no longer U1.PC24
- net DBG_TRACE_SWO: now also U101.PB30; no longer U1.PB30
- net DBG_USB_D+: now also U101.PA25; no longer U1.PA25
- net DBG_USB_D-: now also U101.PA24; no longer U1.PA24
- net DTR_BUS0_AIN0: now also U101.PA2; no longer U1.PA2
- net DTR_BUS0_AIN1: now also U101.PA3; no longer U1.PA3
- net DTR_BUS0_GPIO0: now also U101.PB12; no longer U1.PB12
- net DTR_BUS0_GPIO1: now also U101.PB13; no longer U1.PB13
- net DTR_BUS0_SERCOM0_P0: now also U101.PA8; no longer U1.PA8
- net DTR_BUS0_SERCOM0_P1: now also U101.PA9; no longer U1.PA9
- net DTR_BUS0_SERCOM0_P2: now also U101.PA10; no longer U1.PA10
- net DTR_BUS0_SERCOM0_P3: now also U101.PA11; no longer U1.PA11
- net DTR_BUS1_AIN0: now also U101.PA4; no longer U1.PA4
- net DTR_BUS1_AIN1: now also U101.PA5; no longer U1.PA5
- net DTR_BUS1_GPIO0: now also U101.PB14; no longer U1.PB14
- net DTR_BUS1_GPIO1: now also U101.PB15; no longer U1.PB15
- net DTR_BUS1_SERCOM1_P0: now also U101.PA16; no longer U1.PA16
- net DTR_BUS1_SERCOM1_P1: now also U101.PA17; no longer U1.PA17
- net DTR_BUS1_SERCOM1_P2: now also U101.PA18; no longer U1.PA18
- net DTR_BUS1_SERCOM1_P3: now also U101.PA19; no longer U1.PA19
- net DTR_BUS2_AIN0: now also U101.PC2; no longer U1.PC2
- net DTR_BUS2_AIN1: now also U101.PC3; no longer U1.PC3
- net DTR_BUS2_GPIO0: now also U101.PB16; no longer U1.PB16
- net DTR_BUS2_GPIO1: now also U101.PB17; no longer U1.PB17
- net DTR_BUS2_SERCOM2_P0: now also U101.PA12; no longer U1.PA12
- net DTR_BUS2_SERCOM2_P1: now also U101.PA13; no longer U1.PA13
- net DTR_BUS2_SERCOM2_P2: now also U101.PA14; no longer U1.PA14
- net DTR_BUS2_SERCOM2_P3: now also U101.PA15; no longer U1.PA15
- net DTR_BUS3_AIN0: now also U101.PB4; no longer U1.PB4
- net DTR_BUS3_AIN1: now also U101.PB5; no longer U1.PB5
- net DTR_BUS3_GPIO0: now also U101.PA6; no longer U1.PA6
- net DTR_BUS3_GPIO1: now also U101.PA7; no longer U1.PA7
- net DTR_BUS3_SERCOM7_P0: now also U101.PD8; no longer U1.PD8
- net DTR_BUS3_SERCOM7_P1: now also U101.PD9; no longer U1.PD9
- net DTR_BUS3_SERCOM7_P2: now also U101.PD10; no longer U1.PD10
- net DTR_BUS3_SERCOM7_P3: now also U101.PD11; no longer U1.PD11
- net DTR_DETECT: now also U101.PC31; no longer U1.PC31
- net DTR_MASTER_I2C_SCL: now also U101.PA23, U201.SCL; no longer U1.PA23, U202.SCL
- net DTR_MASTER_I2C_SDA: now also U101.PA22, U201.SDA; no longer U1.PA22, U202.SDA
- net EN_TEMP: now also U101.PC7, U206.ENABLE; no longer U5.ENABLE
- net GND: now also C201.2, C203.2, C204.2, C205.2, J201.1, R204.1, S101.2, U1.GND, U101.GNDANA0, U101.GNDIO0, U101.GNDIO1, U101.GNDIO2, U101.GNDIO3, U101.GNDIO4, U101.GNDIO5, U101.GNDIO6, U101.GNDIO7, U201.GND, U203.AGND, U203.FPWM, U203.PGND, U205.GND; no longer C21.2, C_REG_BIAS.2, C_REG_IN.2, C_REG_OUT.2, J1.B, J1.SHIELD, J1.VSS, J2.1, R4.1, S1.2, U1.GNDANA0, U1.GNDIO0, U1.GNDIO1, U1.GNDIO2, U1.GNDIO3, U1.GNDIO4, U1.GNDIO5, U1.GNDIO6, U1.GNDIO7, U2.AGND, U2.FPWM, U2.PGND, U202.GND, U5.GND
- net LED_B: now also U101.PB28; no longer U1.PB28
- net LED_G: now also U101.PB27; no longer U1.PB27
- net LED_R: now also U101.PB26; no longer U1.PB26
- net N$1: now also U101.VDDCORE; no longer U1.VDDCORE
- net N$13: now also C203.1, U201.REG; no longer C206.1, U202.REG
- net N$2: now also U101.VSW; no longer U1.VSW
- net N$3: now also U101.VDDANA0, U101.VDDANA1; no longer U1.VDDANA0, U1.VDDANA1
- net N$5: now also S101.1; no longer S1.1
- net NRESET: now also U101.NRESET; no longer U1.NRESET
- net VDD_DBG: now also JP_VDBG.2; no longer JP2.2
- net VDD_DBG_JMP: now also JP_VDBG.1, Q204.G, R204.2, U202.P; no longer JP2.1, Q1.G, R4.2, U3.P
- net VREG_BIAS: now also C204.1, U203.BIAS; no longer C_REG_BIAS.1, U2.BIAS
- net VREG_IN: now also C202.1, U201.SYS, U203.EN, U203.IN; no longer C_REG_IN.1, Q1.S, U2.EN, U2.IN, U3.N
- net VREG_LX1: now also L201.1, U203.LX1; no longer L3.1, U2.LX1
- net VREG_LX2: now also L201.2, U203.LX2; no longer L3.2, U2.LX2
- net XIN: now also U101.PB22; no longer U1.PB22
- net XIN32: now also U101.PA0; no longer U1.PA0
- net XOUT: now also U101.PB23; no longer U1.PB23
- net XOUT32: now also U101.PA1; no longer U1.PA1
Other:
- note added: "Current Monitor"
- note added: "Do we lose info about battery by not having the input directly connected to the battery?"
- note added: "External FLASH Storage"
- note added: "Main Battery Supply"
- note removed: "3V7 BATT needs to be included in the debug header so that it can charge the battery from there; no charger on this board"
- note removed: "Battery and Coulomb Counter"
- note removed: "SD Card"
- note removed: "VDD_DBG comes from debug/aux power board. Should be an alternative power source like solar or USB. If charger is on that board, then VDD_DBG should be charger output"
