File: base/Schematics and Boards/CSv2.0_proto/cs_v2.sch (EAGLE design)
At the start: 80 parts, among them J101 J-JTAG-CORTEX-NEEDLE6-LEGS, J301 HIROSE-DF40_44-PIN_CONNECTORS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, J302 HIROSE-DF40_30-PIN_CONNECTORS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, Q201 FK3303010L, Q202 DMG3415UFY4Q-7F, Q203 FK3303010L, Q204 FK3303010L, U101 ATSAMD51, U102 AT25SF641-MHB-T, U201 COULOMB-MAX17262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

Commit message: Rename a few pins to show which SERCOM port is used
Connections:
- net DBG_SERIAL_RX renamed DBG_SERIAL_RX_SERCOM4
- net DBG_SERIAL_TX renamed DBG_SERIAL_TX_SERCOM4
Changed lines of the file:
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@@
 <?xml version="1.0" encoding="utf-8"?>
 <!DOCTYPE eagle SYSTEM "eagle.dtd">
-<eagle version="9.5.2">
+<eagle version="9.6.1">
 <drawing>
 <settings>
@@
 </segment>
 </bus>
-<bus name="DEBUG:CC_IN,DBG_GPIO0,DBG_GPIO1,DBG_GPIO2,DBG_GPIO3,DBG_SERIAL_RX,DBG_SERIAL_TX,DBG_SWCLK,DBG_SWDIO,DBG_SWO,DBG_TRACE_CLK,DBG_TRACE_D0,DBG_TRACE_D1,DBG_TRACE_D2,DBG_TRACE_D3,DBG_TRACE_SWO,DBG_USB_D-,DBG_USB_D+,NRESET,VDD_DBG">
+<bus name="DEBUG:CC_IN,DBG_GPIO0,DBG_GPIO1,DBG_GPIO2,DBG_GPIO3,DBG_SERIAL_RX_SERCOM4,DBG_SERIAL_TX_SERCOM4,DBG_SWCLK,DBG_SWDIO,DBG_SWO,DBG_TRACE_CLK,DBG_TRACE_D0,DBG_TRACE_D1,DBG_TRACE_D2,DBG_TRACE_D3,DBG_TRACE_SWO,DBG_USB_D-,DBG_USB_D+,NRESET,VDD_DBG">
 <segment>
 <wire x1="264.16" y1="22.86" x2="20.32" y2="22.86" width="0.762" layer="92"/>
@@
 </segment>
 </net>
-<net name="DBG_SERIAL_TX" class="0">
+<net name="DBG_SERIAL_TX_SERCOM4" class="0">
 <segment>
 <pinref part="U101" gate="G$1" pin="PB8"/>
@@
 </segment>
 </net>
-<net name="DBG_SERIAL_RX" class="0">
+<net name="DBG_SERIAL_RX_SERCOM4" class="0">
 <segment>
 <pinref part="U101" gate="G$1" pin="PB9"/>
@@
 </segment>
 </bus>
-<bus name="DEBUG:CC_IN,DBG_GPIO0,DBG_GPIO1,DBG_GPIO2,DBG_GPIO3,DBG_SERIAL_RX,DBG_SERIAL_TX,DBG_SWCLK,DBG_SWDIO,DBG_SWO,DBG_TRACE_CLK,DBG_TRACE_D0,DBG_TRACE_D1,DBG_TRACE_D2,DBG_TRACE_D3,DBG_TRACE_SWO,DBG_USB_D-,DBG_USB_D+,NRESET,VDD_DBG">
+<bus name="DEBUG:CC_IN,DBG_GPIO0,DBG_GPIO1,DBG_GPIO2,DBG_GPIO3,DBG_SERIAL_RX_SERCOM4,DBG_SERIAL_TX_SERCOM4,DBG_SWCLK,DBG_SWDIO,DBG_SWO,DBG_TRACE_CLK,DBG_TRACE_D0,DBG_TRACE_D1,DBG_TRACE_D2,DBG_TRACE_D3,DBG_TRACE_SWO,DBG_USB_D-,DBG_USB_D+,NRESET,VDD_DBG">
 <segment>
 <wire x1="215.9" y1="86.36" x2="365.76" y2="86.36" width="0.762" layer="92"/>
@@
 </segment>
 </net>
-<net name="DBG_SERIAL_TX" class="0">
+<net name="DBG_SERIAL_TX_SERCOM4" class="0">
 <segment>
 <wire x1="274.32" y1="86.36" x2="276.86" y2="88.9" width="0.1524" layer="91"/>
@@
 </segment>
 </net>
-<net name="DBG_SERIAL_RX" class="0">
+<net name="DBG_SERIAL_RX_SERCOM4" class="0">
 <segment>
 <wire x1="276.86" y1="86.36" x2="279.4" y2="88.9" width="0.1524" layer="91"/>

Commit message: Add a few signals to DTR card connector
Connections:
- new net DTR_MASTER_IRQ: J301.44
- new net DTR_V_SENSE-: J301.43
Changed lines of the file:
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@@
+</segment>
+</net>
+<net name="DTR_V_SENSE-" class="0">
+<segment>
+<pinref part="J301" gate="G$1" pin="43"/>
+<wire x1="137.16" y1="139.7" x2="137.16" y2="91.44" width="0.1524" layer="91"/>
+<label x="137.16" y="93.98" size="1.778" layer="95" rot="R90"/>
+</segment>
+</net>
+<net name="DTR_MASTER_IRQ" class="0">
+<segment>
+<pinref part="J301" gate="G$1" pin="44"/>
+<wire x1="137.16" y1="160.02" x2="137.16" y2="215.9" width="0.1524" layer="91"/>
+<label x="137.16" y="182.88" size="1.778" layer="95" rot="R90"/>
 </segment>
 </net>
