File: base/Schematics and Boards/CSv2.0_proto/cs_v2.brd (EAGLE design)
At the start: 38.1 x 44.5 mm, 80 parts, among them J101 J-JTAG-CORTEX-NEEDLE6-LEGS, J301 HIROSE-DF40_44-PIN_CONNECTORS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, J302 HIROSE-DF40_30-PIN_CONNECTORS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, Q201 FK3303010L, Q202 DMG3415UFY4Q-7F, Q203 FK3303010L, Q204 FK3303010L, U101 ATSAMD51, U102 AT25SF641-MHB-T, U201 COULOMB-MAX17262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

Commit message: Rename a few pins to show which SERCOM port is used
Connections:
- net DBG_SERIAL_RX renamed DBG_SERIAL_RX_SERCOM4
- net DBG_SERIAL_TX renamed DBG_SERIAL_TX_SERCOM4
Changed lines of the file:
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@@
 <?xml version="1.0" encoding="utf-8"?>
 <!DOCTYPE eagle SYSTEM "eagle.dtd">
-<eagle version="9.5.2">
+<eagle version="9.6.1">
 <drawing>
 <settings>
@@
 <wire x1="22.3266" y1="34.1884" x2="22.1917875" y2="34.3232125" width="0.1016" layer="15"/>
 </signal>
-<signal name="DBG_SERIAL_TX">
+<signal name="DBG_SERIAL_TX_SERCOM4">
 <contactref element="U101" pad="PB08"/>
 <contactref element="TXDBG" pad="TP"/>
@@
 <via x="20.1422" y="40.513" extent="1-16" drill="0.1524" alwaysstop="yes"/>
 </signal>
-<signal name="DBG_SERIAL_RX">
+<signal name="DBG_SERIAL_RX_SERCOM4">
 <contactref element="U101" pad="PB09"/>
 <contactref element="RXDBG" pad="TP"/>

Commit message: Add a few signals to DTR card connector
Connections:
- new net DTR_MASTER_IRQ: J301.44
- new net DTR_V_SENSE-: J301.43
Changed lines of the file:
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@@
 <wire x1="28.1432" y1="30.2768" x2="28.1432" y2="22.7076" width="0.1016" layer="16"/>
+</signal>
+<signal name="DTR_V_SENSE-">
+<contactref element="J301" pad="43"/>
+</signal>
+<signal name="DTR_MASTER_IRQ">
+<contactref element="J301" pad="44"/>
 </signal>
 </signals>
