File: debug/Schematics and Boards/cs_debug/cs_debug_v1.sch (EAGLE design)
At the start: 59 parts, among them J401 J-USB-HIROSE-MICRO-USB, Y101 32.768kHz, Y102 12mHz-12pF-K7

Commit message: Add amplifiers and passives for high-side current monitor
FETs still to be added. Haven't set values on passives or added any part numbers to the circuit. Still need to convert the whole thing into a group. The nets have been named, and a few notes left behind for the remaining task
Parts:
- added C1: (no value), Capacitors:C-0402
- added R1, R2, R3, R4, R5, R6, R7, R8: (no value), Resistors:R-0402
- added U1: INA225AIDGK, Amplifiers:INA225AIDGK
- added U2: OPA357AIDBVTG4, Amplifiers:OPA357AIDBVTG4
Connections:
- new net AGND: R5.1, U1.REF, U1.V-, U2.V-
- new net DCBIAS_SHUTDOWN: R6.1
- new net DIFFAMP_GAIN0: U1.GS0
- new net DIFFAMP_GAIN1: U1.GS1
- new net N$1: R1.2, R2.2, U2.IN+
- new net N$3: U1.OUT
- new net N$4: R3.1, U2.ENABLE
- new net N$6: R4.1, R5.2, U2.IN-
- new net N$7: R4.2, R7.1, U2.OUT
- new net N$8: C1.2, R8.2, U1.IN+
- new net N$9: C1.1, R7.2, U1.IN-
- new net V_OFFSET_IN: R1.1
- new net V_SENSE_N: R2.1
- new net V_SENSE_P: R8.1
- net 3V3_INSTR_PROC: now also R3.2, R6.2, U1.V+, U2.V+
Other:
- note added: "High-Side Current Monitor"
- note added: "Instrumentation Processor"
- note added: "NFET to handle control signal, driven by instrumentation proc pin"
- note added: "PFET to disable and opamp and connect VSENSE- to OUT"
- note added: "this input signal should be driven low by default to keep opamp enabled"

Commit message: Add high side current monitors as groups; label pins from main connector
Parts:
- removed C1: (no value), Capacitors:C-0402
- removed J_DEBUG_MAIN_HEADER: HIROSE-DF40_30-PIN_CONNECTORS-HEADER, Connectors:HIROSE-DF40_30-PIN_CONNECTORS-HEADER
- removed R1, R2, R3, R4, R5, R6, R7, R8: (no value), Resistors:R-0402
- removed U1: INA225AIDGK, Amplifiers:INA225AIDGK
- removed U2: OPA357AIDBVTG4, Amplifiers:OPA357AIDBVTG4
- added C10, C13, C4, C7: 68p, Capacitors:C-0402
- added C11, C12, C14, C15, C5, C6, C8, C9: 0.1u, Capacitors:C-0402
- added JP1, JP2, JP3, JP4: JUMPER-SMT_2_NC_PASTE_NO-SILK, SparkFun-Jumpers:JUMPER-SMT_2_NC_PASTE_NO-SILK
- added J_DEBUG_TO_MAIN_HEADER: HIROSE-DF40_30-PIN_CONNECTORS-HEADER, Connectors:HIROSE-DF40_30-PIN_CONNECTORS-HEADER
- added Q10, Q4, Q6, Q8: 2N7002P, Switches:2N7002P
- added Q3, Q5, Q7, Q9: FDN340P, Switches:FDN340P
- added R10, R12, R14, R18, R20, R22, R26, R28, R30, R34, R36, R38: 10k, Resistors:R-0402
- added R11, R19, R27, R35: 100k, Resistors:R-0402
- added R13, R17, R21, R25, R29, R33, R37, R9: 249k, Resistors:R-0402
- added R15, R16, R23, R24, R31, R32, R39, R40: 5.1, Resistors:R-0603
- added U10, U4, U6, U8: OPA357AIDBVTG4, Amplifiers:OPA357AIDBVTG4
- added U3, U5, U7, U9: INA225AIDGK, Amplifiers:INA225AIDGK
Connections:
- removed net DCBIAS_SHUTDOWN: R6.1
- removed net DIFFAMP_GAIN0: U1.GS0
- removed net DIFFAMP_GAIN1: U1.GS1
- removed net N$1: R1.2, R2.2, U2.IN+
- removed net N$3: U1.OUT
- removed net N$4: R3.1, U2.ENABLE
- removed net N$6: R4.1, R5.2, U2.IN-
- removed net N$7: R4.2, R7.1, U2.OUT
- removed net N$8: C1.2, R8.2, U1.IN+
- removed net N$9: C1.1, R7.2, U1.IN-
- removed net V_OFFSET_IN: R1.1
- removed net V_SENSE_N: R2.1
- new net CM_DTR_DCBIAS_SHUTDOWN: Q8.GATE, R30.1
- new net CM_DTR_DIFFAMP_GAIN0: U7.GS0
- new net CM_DTR_DIFFAMP_GAIN1: U7.GS1
- new net CM_DTR_DIFFAMP_N3: C10.1, R31.2, U7.IN-
- new net CM_DTR_DIFFAMP_OUT: U7.OUT
- new net CM_DTR_DIFFAMP_P3: C10.2, R32.2, U7.IN+
- new net CM_DTR_OPAMP_ENABLE3: Q7.G, Q8.DRAIN, R27.1, U8.ENABLE
- new net CM_DTR_OPAMP_N3: R28.1, R29.2, U8.IN-
- new net CM_DTR_OPAMP_OUT3: Q7.S, R28.2, R31.1, U8.OUT
- new net CM_DTR_OPAMP_P3: R25.2, R26.2, U8.IN+
- new net CM_DTR_V_OFFSET_IN: R25.1
- new net CM_DTR_V_SENSE_N: J_DEBUG_TO_MAIN_HEADER.16, Q7.D, R26.1
- new net CM_DTR_V_SENSE_P: JP4.2, R32.1
- new net CM_PROC_DCBIAS_SHUTDOWN: Q4.GATE, R14.1
- new net CM_PROC_DIFFAMP_GAIN0: U3.GS0
- new net CM_PROC_DIFFAMP_GAIN1: U3.GS1
- new net CM_PROC_DIFFAMP_N1: C4.1, R15.2, U3.IN-
- new net CM_PROC_DIFFAMP_OUT: U3.OUT
- new net CM_PROC_DIFFAMP_P1: C4.2, R16.2, U3.IN+
- new net CM_PROC_OPAMP_ENABLE1: Q3.G, Q4.DRAIN, R11.1, U4.ENABLE
- new net CM_PROC_OPAMP_N1: R12.1, R13.2, U4.IN-
- new net CM_PROC_OPAMP_OUT1: Q3.S, R12.2, R15.1, U4.OUT
- new net CM_PROC_V_OFFSET_IN: R9.1
- new net CM_PROC_V_SENSE_N: J_DEBUG_TO_MAIN_HEADER.14, Q3.D, R10.1
- new net CM_PROC_V_SENSE_P: JP1.2, R16.1
- new net CM_STORAGE_DCBIAS_SHUTDOWN: Q6.GATE, R22.1
- new net CM_STORAGE_DIFFAMP_GAIN0: U5.GS0
- new net CM_STORAGE_DIFFAMP_GAIN1: U5.GS1
- new net CM_STORAGE_DIFFAMP_N1: C7.1, R23.2, U5.IN-
- new net CM_STORAGE_DIFFAMP_OUT: U5.OUT
- new net CM_STORAGE_DIFFAMP_P1: C7.2, R24.2, U5.IN+
- new net CM_STORAGE_OPAMP_ENABLE1: Q5.G, Q6.DRAIN, R19.1, U6.ENABLE
- new net CM_STORAGE_OPAMP_N1: R20.1, R21.2, U6.IN-
- new net CM_STORAGE_OPAMP_OUT1: Q5.S, R20.2, R23.1, U6.OUT
- new net CM_STORAGE_OPAMP_P1: R17.2, R18.2, U6.IN+
- new net CM_STORAGE_V_OFFSET_IN: R17.1
- new net CM_STORAGE_V_SENSE_N: J_DEBUG_TO_MAIN_HEADER.18, Q5.D, R18.1
- new net CM_STORAGE_V_SENSE_P: JP2.2, R24.1
- new net CM_TEMP_DCBIAS_SHUTDOWN: Q10.GATE, R38.1
- new net CM_TEMP_DIFFAMP_GAIN0: U9.GS0
- new net CM_TEMP_DIFFAMP_GAIN1: U9.GS1
- new net CM_TEMP_DIFFAMP_N1: C13.1, R39.2, U9.IN-
- new net CM_TEMP_DIFFAMP_OUT: U9.OUT
- new net CM_TEMP_DIFFAMP_P1: C13.2, R40.2, U9.IN+
- new net CM_TEMP_OPAMP_ENABLE1: Q10.DRAIN, Q9.G, R35.1, U10.ENABLE
- new net CM_TEMP_OPAMP_N1: R36.1, R37.2, U10.IN-
- new net CM_TEMP_OPAMP_OUT1: Q9.S, R36.2, R39.1, U10.OUT
- new net CM_TEMP_OPAMP_P1: R33.2, R34.2, U10.IN+
- new net CM_TEMP_V_OFFSET_IN: R33.1
- new net CM_TEMP_V_SENSE_N: J_DEBUG_TO_MAIN_HEADER.20, Q9.D, R34.1
- new net CM_TEMP_V_SENSE_P: JP3.2, R40.1
- new net CM__PROCOPAMP_P1: R10.2, R9.2, U4.IN+
- new net MAIN_GPIO0: J_DEBUG_TO_MAIN_HEADER.7
- new net MAIN_GPIO1: J_DEBUG_TO_MAIN_HEADER.9
- new net MAIN_GPIO2: J_DEBUG_TO_MAIN_HEADER.11
- new net MAIN_GPIO3: J_DEBUG_TO_MAIN_HEADER.13
- new net MAIN_NRESET: J_DEBUG_TO_MAIN_HEADER.30
- new net MAIN_SWD_SWCLK: J_DEBUG_TO_MAIN_HEADER.19
- new net MAIN_SWD_SWDIO: J_DEBUG_TO_MAIN_HEADER.21
- new net MAIN_TRACE_CLK: J_DEBUG_TO_MAIN_HEADER.26
- new net MAIN_TRACE_D0: J_DEBUG_TO_MAIN_HEADER.23
- new net MAIN_TRACE_D1: J_DEBUG_TO_MAIN_HEADER.25
- new net MAIN_TRACE_D2: J_DEBUG_TO_MAIN_HEADER.27
- new net MAIN_TRACE_D3: J_DEBUG_TO_MAIN_HEADER.29
- new net MAIN_TRACE_SWO: J_DEBUG_TO_MAIN_HEADER.28
- new net MAIN_USART_RX: J_DEBUG_TO_MAIN_HEADER.17
- new net MAIN_USART_TX: J_DEBUG_TO_MAIN_HEADER.15
- new net MAIN_USB_DATA_N: J_DEBUG_TO_MAIN_HEADER.22
- new net MAIN_USB_DATA_P: J_DEBUG_TO_MAIN_HEADER.24
- new net VDD_TO_MAIN: J_DEBUG_TO_MAIN_HEADER.2, J_DEBUG_TO_MAIN_HEADER.4
- new net V_BATT_MAIN: J_DEBUG_TO_MAIN_HEADER.10, J_DEBUG_TO_MAIN_HEADER.6, J_DEBUG_TO_MAIN_HEADER.8
- net 3V3_INSTR_PROC: now also C11.1, C12.1, C14.1, C15.1, C5.1, C6.1, C8.1, C9.1, R11.2, R14.2, R19.2, R22.2, R27.2, R30.2, R35.2, R38.2, U10.V+, U3.V+, U4.V+, U5.V+, U6.V+, U7.V+, U8.V+, U9.V+; no longer R3.2, R6.2, U1.V+, U2.V+
- net AGND: now also C11.2, C12.2, C14.2, C15.2, C5.2, C6.2, C8.2, C9.2, Q10.SOURCE, Q4.SOURCE, Q6.SOURCE, Q8.SOURCE, R13.1, R21.1, R29.1, R37.1, U10.V-, U3.REF, U3.V-, U4.V-, U5.REF, U5.V-, U6.V-, U7.REF, U7.V-, U8.V-, U9.REF, U9.V-; no longer R5.1, U1.REF, U1.V-, U2.V-
- net DGND: now also J_DEBUG_TO_MAIN_HEADER.1, J_DEBUG_TO_MAIN_HEADER.3, J_DEBUG_TO_MAIN_HEADER.5
- net V_SENSE_P: now also JP1.1, JP2.1, JP3.1, JP4.1, J_DEBUG_TO_MAIN_HEADER.12; no longer R8.1
Other:
- note added: "A pun on temporary and temperature It is probably unnecessary to dedicate an entire channel to the temperature sensor, whose current draw is near negligible Instead, we may change this channel to be used for something else, most likely another signal from the daughter card"
- note added: "Debug to Main board connector"
- note added: "High-Side Current Monitors"
- note added: "N-ch MOSFET to enable (gate low) or disable (gate high) OPAMP Summing Circuit. If disable, bypass opamp using PFET. Pullup on gate defaults to bypassing the opamp"
- note added: "Trace signals may be reused as GPIOs; they require a special debugger, but allow in-depth debugging"
- note removed: "High-Side Current Monitor"
- note removed: "NFET to handle control signal, driven by instrumentation proc pin"
- note removed: "PFET to disable and opamp and connect VSENSE- to OUT"

Commit message: Add LDOs, update formatting
Parts:
- added C1, C2: 10u, Capacitors:C-0805
- added C205: 22u, Capacitors:C-0805
- added C3: 0.1u, Capacitors:C-0402
- added JP5, JP6: JUMPER-SMT_2_NC_PASTE_NO-SILK, SparkFun-Jumpers:JUMPER-SMT_2_NC_PASTE_NO-SILK
- added U1: AP2120N-3.3TRG1, Regulators:AP2120N
- added U2: TLV1117LV33DCYR, Regulators:TLV1117LV33DCYR
Connections:
- new net 3V3_INSTR_MEAS: C1.1, C11.1, C12.1, C14.1, C15.1, C5.1, C6.1, C8.1, C9.1, R11.2, R14.2, R19.2, R22.2, R27.2, R30.2, R35.2, R38.2, U1.OUT, U10.V+, U3.V+, U4.V+, U5.V+, U6.V+, U7.V+, U8.V+, U9.V+
- new net N$1: JP5.2, U1.IN
- new net N$3: C205.1, C3.1, JP5.1, JP6.1
- new net N$4: JP6.2, U2.IN
- new net N$6: U_INSTR_PROC.PB28
- new net N$7: U_INSTR_PROC.PB29
- new net N$8: U_INSTR_PROC.PB30
- new net N$9: U_INSTR_PROC.PB31
- net 3V3_INSTR_PROC: now also C2.1, U2.OUT; no longer C11.1, C12.1, C14.1, C15.1, C5.1, C6.1, C8.1, C9.1, R11.2, R14.2, R19.2, R22.2, R27.2, R30.2, R35.2, R38.2, U10.V+, U3.V+, U4.V+, U5.V+, U6.V+, U7.V+, U8.V+, U9.V+
- net AGND: now also C1.2, U1.GND
- net DGND: now also C2.2, C205.2, C3.2, U2.GND
Other:
- note added: "Add battery charger w/ switch on output Include a switch to disconnect charger output from voltage that goes to regulator on main board"
- note added: "Computation and Communication Structures Group"
- moved on the sheet: C10, C101, C102, C103, C104, C105, C106, C107, C108, C109, C11, C110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

Commit message: Signals from instrumentation processor to current monitors
Parts:
- removed LED101: RED, adafruit:LEDCHIPLED_0603
- removed LED102: GREEN, adafruit:LEDCHIPLED_0603
- removed R107, R108: 1k, Resistors:R-0603
- added R1: 0, Resistors:R-2010
Connections:
- net D+ renamed INSTR_PROC_USB_D_P
- net D- renamed INSTR_PROC_USB_D_N
- net MAIN_TRACE_D2 renamed MAIN_TRACE_D2/GPIO8
- net MAIN_TRACE_D3 renamed MAIN_TRACE_D3/GPIO9
- removed net CM_PROC_V_OFFSET_IN: R9.1
- removed net MAIN_TRACE_CLK: J_DEBUG_TO_MAIN_HEADER.26
- removed net MAIN_TRACE_D0: J_DEBUG_TO_MAIN_HEADER.23
- removed net MAIN_TRACE_D1: J_DEBUG_TO_MAIN_HEADER.25
- removed net MAIN_TRACE_SWO: J_DEBUG_TO_MAIN_HEADER.28
- removed net N$31: LED101.A, R107.1
- removed net USR_LED_GREEN: LED102.C
- removed net USR_LED_RED: LED101.C
- new net INSTR_PROC_USART_RX: U_INSTR_PROC.PD5
- new net INSTR_PROC_USART_TX: U_INSTR_PROC.PD4
- new net MAIN_TRACE_CLK/GPIO4: J_DEBUG_TO_MAIN_HEADER.26, U_INSTR_PROC.PC15
- new net MAIN_TRACE_D0/GPIO6: J_DEBUG_TO_MAIN_HEADER.23, U_INSTR_PROC.PB1
- new net MAIN_TRACE_D1/GPIO7: J_DEBUG_TO_MAIN_HEADER.25, U_INSTR_PROC.PB2
- new net MAIN_TRACE_SWO/GPIO5: J_DEBUG_TO_MAIN_HEADER.28, U_INSTR_PROC.PB0
- new net N$10: U_INSTR_PROC.PB13
- new net N$11: U_INSTR_PROC.PA2
- net 3V3_INSTR_PROC: no longer R107.2, R108.2
- net AGND: now also R1.2
- net CM_DTR_DCBIAS_SHUTDOWN: now also U_INSTR_PROC.PD2
- net CM_DTR_DIFFAMP_GAIN0: now also U_INSTR_PROC.PC6
- net CM_DTR_DIFFAMP_GAIN1: now also U_INSTR_PROC.PC5
- net CM_DTR_DIFFAMP_OUT: now also U_INSTR_PROC.PA6
- net CM_PROC_DCBIAS_SHUTDOWN: now also U_INSTR_PROC.PD3
- net CM_PROC_DIFFAMP_GAIN0: now also U_INSTR_PROC.PC8
- net CM_PROC_DIFFAMP_GAIN1: now also U_INSTR_PROC.PC7
- net CM_PROC_DIFFAMP_OUT: now also U_INSTR_PROC.PA16
- net CM_STORAGE_DCBIAS_SHUTDOWN: now also U_INSTR_PROC.PD1
- net CM_STORAGE_DIFFAMP_GAIN0: now also U_INSTR_PROC.PC4
- net CM_STORAGE_DIFFAMP_GAIN1: now also U_INSTR_PROC.PC3
- net CM_STORAGE_DIFFAMP_OUT: now also U_INSTR_PROC.PA4
- net CM_TEMP_DCBIAS_SHUTDOWN: now also U_INSTR_PROC.PD0
- net CM_TEMP_DIFFAMP_GAIN0: now also U_INSTR_PROC.PC2
- net CM_TEMP_DIFFAMP_GAIN1: now also U_INSTR_PROC.PC1
- net CM_TEMP_DIFFAMP_OUT: now also U_INSTR_PROC.PA3
- net DGND: now also R1.1
- net MAIN_GPIO0: now also U_INSTR_PROC.PC19
- net MAIN_GPIO1: now also U_INSTR_PROC.PC18
- net MAIN_GPIO2: now also U_INSTR_PROC.PC17
- net MAIN_GPIO3: now also U_INSTR_PROC.PC16
- net N$3: now also U_INSTR_PROC.PB11; no longer C205.1, C3.1, JP5.1, JP6.1
- net N$5: now also U_INSTR_PROC.PB12; no longer LED102.A, R108.1
- net VDD_TO_MAIN: now also C205.1, C3.1, JP5.1, JP6.1
Other:
- note added: "All analog signals should be routed between the GND domains underneath this resistor"
- note added: "JTAG lines"
- note added: "May need to use a larger resistor (2512) because there are plenty of analog signals There are >=9 analog signals 1 for vense+ 4 for sense- 4 for DAC outputs"
- note added: "Supposedly used to communicate between main and instr processors"
- note added: "What is this for on powerdue?"
- moved on the sheet: C1, C10, C11, C12, C120, C121, C122, C123, C125, C127, C128, C2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

Commit message: Add debug connectors, DAC, pull-ups to schematic
Parts:
- added C16: 0.1u, Capacitors:C-0402
- added J1, J2: J-JTAG-CORTEX_SMD, Connectors:J-JTAG-CORTEX_SMD
- added J3: J-JTAG-CORTEX-NEEDLE6-LEGS, Connectors:J-JTAG-CORTEX-NEEDLE6-LEGS
- added JP7: JUMPER-SMT_2_NC_PASTE_NO-SILK, SparkFun-Jumpers:JUMPER-SMT_2_NC_PASTE_NO-SILK
- added R2, R3, R6: 100k, Resistors:R-0402
- added R4, R5: 4.7k, Resistors:R-0402
- added U11: DAC7574IDGS, DACs:DAC7574IDGS
Connections:
- removed net CPU_RESET: C119.2, S101.2, U_INSTR_PROC.NRSTB
- removed net N$10: U_INSTR_PROC.PB13
- removed net N$3: U_INSTR_PROC.PB11
- removed net N$5: U_INSTR_PROC.PB12
- removed net N$6: U_INSTR_PROC.PB28
- removed net N$7: U_INSTR_PROC.PB29
- removed net N$8: U_INSTR_PROC.PB30
- removed net N$9: U_INSTR_PROC.PB31
- removed net UOTGID: J401.USBID, VR401.1
- new net CM_PROC_V_OFFSET_IN: U11.VOUTA
- new net INSTR_PROC_I2C_SCL: R4.2, U11.SCL, U_INSTR_PROC.PB13
- new net INSTR_PROC_I2C_SDA: R5.2, U11.SDA, U_INSTR_PROC.PB12
- new net INSTR_PROC_JTAG_TCK/SWCLK: J2.SWDCLK/TCK, J3.SWCLK, R3.1, U_INSTR_PROC.PB28
- new net INSTR_PROC_JTAG_TDI: J2.NC/TDI, R6.1, U_INSTR_PROC.PB29
- new net INSTR_PROC_JTAG_TDO/SWO: J2.SWO/TDO, J3.SWO, U_INSTR_PROC.PB30
- new net INSTR_PROC_JTAG_TMS/SWDIO: J2.SWDIO/TMS, J3.SWDIO, R2.1, U_INSTR_PROC.PB31
- new net INSTR_PROC_NRESET: C119.2, J2.!RESET, J3.NRESET, S101.2, U_INSTR_PROC.NRSTB
- new net INSTR_PROC_USB_UOTGID: J401.USBID, U_INSTR_PROC.PB11, VR401.1
- new net N$12: C205.1, C3.1, JP5.1, JP6.1, JP7.1
- net 3V3_INSTR_MEAS: now also C16.1, U11.VDD
- net 3V3_INSTR_PROC: now also J2.VCC, J3.VTREF, R2.2, R3.2, R4.1, R5.1, R6.2
- net AGND: now also C16.2, U11.A0, U11.A1, U11.GND
- net CM_DTR_V_OFFSET_IN: now also U11.VOUTB
- net CM_STORAGE_V_OFFSET_IN: now also U11.VOUTC
- net CM_TEMP_V_OFFSET_IN: now also U11.VOUTD
- net DGND: now also J1.GND@3, J1.GND@5, J2.GND@3, J2.GND@5, J2.GNDDTCT, J3.GND
- net MAIN_NRESET: now also J1.!RESET
- net MAIN_SWD_SWCLK: now also J1.SWDCLK/TCK
- net MAIN_SWD_SWDIO: now also J1.SWDIO/TMS
- net VDD_TO_MAIN: now also JP7.2; no longer C205.1, C3.1, JP5.1, JP6.1
- net V_SENSE_P: now also J1.VCC
Other:
- note added: "5x2 0.05'' JTAG connector (Main)"
- note added: "Both debug connector options in case dev is missing a cable. Tag-connect is missing TDI, so it may not work"
- note added: "Channel 0"
- note added: "Channel 1"
- note added: "Channel 2"
- note added: "Channel 3"
- note added: "pullups are present on main board"
- note removed: "JTAG lines"
- moved on the sheet: C1, C10, C11, C12, C13, C14, C15, C2, C205, C3, C4, C401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

Commit message: Finish first-pass of Debug Board schematic
Parts:
- removed C104, C105, C109, C110, C111, C112, C113, C114, C116, C117, C121, C122, C123, C124, C125, C127, C128: 0.1uF, Capacitors:C-0603
- removed C119: 10nF, Capacitors:C-0603
- removed R104, R106: 100k, Resistors:R-0603
- removed S101: Momentary, Switches:MOMENTARY-SWITCH-SPST-SMD-5.2-REDUNDANT
- added C18, C208: 4.7u, Capacitors:C-0402
- added C20, C28: 10n, Capacitors:C-0402
- added C21: 22u, Capacitors:C-0805
- added C22, C29, C30, C31, C32, C33, C34, C35, C36, C37, C38, C39, C40, C41, C42, C43, C44: 0.1u, Capacitors:C-0402
- added D1: MBR120VLSFT3GOSCT-ND, adafruit:DIODESOD-123
- added F2: MF-MSMF050-2, adafruit:PTCFUSE-1812
- added J19: Solar, Connectors:J-JST2-SMT-RA
- added JMP_LOG: (no value), Connectors:J-03
- added JP10: JUMPER-SMT_2_NC_PASTE_NO-SILK, SparkFun-Jumpers:JUMPER-SMT_2_NC_PASTE_NO-SILK
- added JP11: JUMPER-SMT_3_1-NC_PASTE_NO-SILK, Connectors:JUMPER-SMT_3_1-NC_PASTE_NO-SILK
- added JP12, JP8, JP9: JUMPER-SMT_2_NC_PASTE_NO-SILK, Connectors:JUMPER-SMT_2_NC_PASTE_NO-SILK
- added L1: 3.3µH/±20%/450mA, SparkFun-Coils:INDUCTOR-0805-3.3UH
- added R201: 270k, Resistors:R-0402
- added R202, R204, R41, R8: 100k, Resistors:R-0402
- added R203: 2k, Resistors:R-0402
- added R206, R7: 10k, Resistors:R-0402
- added S1: Momentary, Switches:SW_EVQ-P7L01P_SPST_RA
- added S201: (no value), Switches:SLIDESWITCH-SPDT-SMD-RIGHT-ANGLE
- added U12: MCP73871T-2CCI/ML, Chargers:MCP73871T-2CCI/ML
- C103, C107, C17, C19: MPN (none) -> C0603C160J5GACTU; PART_NO (none) -> C0603C160J5GACTU
- C108: MPN (none) -> C0603C100K8RAC7867; PART_NO (none) -> C0603C100K8RAC7867
- C11, C12, C14, C15, C3, C5, C6, C8, C9: MPN (none) -> C0402C104K8RACTU
- C205: MPN (none) -> C0805C226M8PAC7800
- C23, C24, C25, C26, C27: value 22uF -> 22u; MPN (none) -> C0805C226M8PAC7800; PART_NO (none) -> C0805C226M8PAC7800; TC (none) -> X5R; VOLTAGE (none) -> 10V
- C401: device Capacitors:C-0805 -> Capacitors:C-0402; MPN (none) -> C0402C225M8PACTU; PART_NO (none) -> C0402C225M8PACTU
- J401: PART_NO (none) -> ZX62D-AB-5P8(30)
- J_DEBUG_TO_MAIN_HEADER: MPN (none) -> DF40C-30DP-0.4V(51); PART_NO (none) -> DF40C-30DP-0.4V(51)
- L101, L102: PART_NO (none) -> MH2029-300Y
- L103, L104: PART_NO (none) -> MH2029-300Y; SPICEPREFIX (none) -> L
- R101, R102: device Resistors:R-0603 -> Resistors:R-0402; MPN (none) -> ERJ-2GEJ390X; PART_NO (none) -> ERJ-2GEJ390X
- R103: device Resistors:R-0603 -> Resistors:R-0402; MPN (none) -> ERJ-2GEJ682X; PART_NO (none) -> ERJ-2GEJ682X
- R2, R3, R6: PART_NO (none) -> ERJ-2GEJ104X
- R4, R5: MPN (none) -> ERJ-2GEJ472X
- S102: device Switches:MOMENTARY-SWITCH-SPST-SMD-5.2-REDUNDANT -> Switches:SW_EVQ-P7L01P_SPST_RA; DESCRIPTION Erase -> (none); MPN (none) -> EVQP7L01P
- VR401, VR402, VR403: PART_NO (none) -> CG0603MLC-05E
- Y101: PART_NO (none) -> ECS-.327-12.5-34B-TR
- Y102: PART_NO (none) -> ABM8G-12.000MHZ-4Y-T3
- renumbered C101 to C27, C102 to C17, C106 to C19, C115 to C26, C118 to C25, C120 to C23, C126 to C24
Connections:
- removed net INSTR_PROC_USART_RX: U_INSTR_PROC.PD5
- removed net INSTR_PROC_USART_TX: U_INSTR_PROC.PD4
- removed net N$12: C205.1, C3.1, JP5.1, JP6.1, JP7.1
- removed net VUSB: C401.1, J401.VBUS
- new net BAT_CHG_PROG1: R203.2, U12.PROG1
- new net CHG_VPCC: R201.1, R202.2, U12.VPCC
- new net EXT_VIN: D1.A, J19.2
- new net GND: C18.2, C208.2, J19.1, S1.1
- new net INSTR_PROC_NRESET_SW: C28.2, JP12.2, S1.2, U_INSTR_PROC.NRSTB
- new net N$10: R204.2, U12.PROG3
- new net N$3: JP8.2, U_INSTR_PROC.PD5
- new net N$5: JP9.2, U_INSTR_PROC.PD4
- new net N$6: L1.2, S201.P
- new net N$8: F2.2, U12.VBAT, U12.VBAT_SENSE
- new net THERM: R206.2, U12.THERM
- new net VCHRG_BATT: C18.1, F2.1, JP10.1
- new net VCHRG_OUT: C208.1, JP11.3, U12.OUT
- new net VREG_IN: C205.1, C3.1, JP11.2, JP5.1, JP6.1, JP7.1
- new net VSRC_RAW: JP11.1, R201.2, S201.S, U12.!TE, U12.CE, U12.IN, U12.PROG2, U12.SEL
- net 3V3_INSTR_PROC: now also C28.1, C37.1, C38.1, C39.1, C40.1, C41.1, C42.1, R41.1; no longer C104.1, C105.1, C109.1, C110.1, C111.1, C112.1, C119.1, R106.2
- net ADVREF: now also C29.1; no longer C116.1
- net ADVREF_PRE: now also C22.1; no longer C114.1
- net CM_PROC_V_OFFSET_IN: now also R9.1
- net DGND: now also C20.2, C21.2, C22.2, C29.2, C30.2, C31.2, C32.2, C33.2, C34.2, C35.2, C36.2, C37.2, C38.2, C39.2, C40.2, C41.2, C42.2, C43.2, C44.2, JMP_LOG.3, R202.1, R203.1, R204.1, R206.1, R7.1, R8.2, U12.EP, U12.VSS; no longer C104.2, C105.2, C109.2, C110.2, C111.2, C112.2, C113.2, C114.2, C116.2, C117.2, C121.2, C122.2, C123.2, C124.2, C125.2, C127.2, C128.2, R104.1, S101.1
- net FWUP: now also R41.2; no longer R106.1
- net INSTR_PROC_NRESET: now also JP12.1; no longer C119.2, S101.2, U_INSTR_PROC.NRSTB
- net MAIN_USART_RX: now also JMP_LOG.1, JP8.1
- net MAIN_USART_TX: now also JMP_LOG.2, JP9.1
- net TST: now also R8.1; no longer R104.2
- net VBUS: now also C20.1, C21.1, C401.1, D1.C, J401.VBUS, L1.1, R7.2
- net VDDANA1: now also C44.1; no longer C117.1
- net VDDOUT: now also C30.1, C31.1, C32.1, C33.1, C34.1, C35.1; no longer C121.1, C122.1, C123.1, C125.1, C127.1, C128.1
- net VDDOUTMI: now also C43.1; no longer C113.1
- net VDDPLL: now also C36.1; no longer C124.1
- net V_BATT_MAIN: now also JP10.2
Other:
- note added: "Add USB port for the main board? Data lines for D51 are present here Would we need a power switch/combiner?"
- note added: "Charger"
- note added: "Erase"
- note added: "GND Bridge"
- note added: "Instrumentation Processor Debugging"
- note added: "Power Sources and USB"
- note added: "Power switch"
- note added: "Regulators"
- note added: "Reset"
- note added: "USART lines between processors??"
- note removed: "Add battery charger w/ switch on output Include a switch to disconnect charger output from voltage that goes to regulator on main board"
- note removed: "Supposedly used to communicate between main and instr processors"
- moved on the sheet: C1, C16, C2, C205, C3, C401, J401, JP5, JP6, JP7, R1, R21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

Commit message: Change USART Header on debug board
Parts:
- removed JMP_LOG: (no value), Connectors:J-03
- added C45: 2.2uF, Capacitors:C-0805
- added J4: J-SERIAL-PORT, Connectors:J-SERIAL-PORT
- added J403: J-WURTH-USBC, Connectors:J-WURTH-USBC
- added JP13: JUMPER-SMT_2_NC_PASTE_NO-SILK, Connectors:JUMPER-SMT_2_NC_PASTE_NO-SILK
- added R422, R423: 5.1k, Resistors:R-0603
- added VR1, VR2: VARISTOR, Diodes:VARISTOR
Connections:
- new net CC1: J403_CONNECTOR.CC1, R422.2
- new net CC2: J403_CONNECTOR.CC2, R423.2
- new net D+: J403_CONNECTOR.DP1, J403_CONNECTOR.DP2, VR1.1
- new net D-: J403_CONNECTOR.DN1, J403_CONNECTOR.DN2, VR2.1
- new net UCTX_DBGRX: J403_CONNECTOR.SBU1, J403_CONNECTOR.SBU2
- net 3V3_INSTR_PROC: now also JP13.1
- net DGND: now also J4.GND; no longer JMP_LOG.3
- net GND: now also C45.2, J403_CONNECTOR.GND, J403_CONNECTOR.GND1, J403_CONNECTOR.GND2, J403_CONNECTOR.GND3, J403_SHIELD.SHIELD, R422.1, R423.1, VR1.2, VR2.2
- net MAIN_USART_RX: now also J4.TX-O; no longer JMP_LOG.1
- net MAIN_USART_TX: now also J4.RX-I; no longer JMP_LOG.2
- net N$11: now also J4.VCC-I, JP13.2; no longer U_INSTR_PROC.PA2
- net VBUS: now also C45.1, J403_CONNECTOR.VBUS, J403_CONNECTOR.VBUS1, J403_CONNECTOR.VBUS2, J403_CONNECTOR.VBUS3
Other:
- note added: "10x cap for larger RC constant"
- note added: "Switch to USB type-c and include a hub IC to provide power, data lines to each"
- note removed: "Add USB port for the main board? Data lines for D51 are present here Would we need a power switch/combiner?"
- note removed: "USART lines between processors??"
- note removed: "What is this for on powerdue?"
- moved on the sheet: C1, C18, C2, C205, C208, C3, D1, F2, J19, JP11, JP5, JP6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
