File: debug/Schematics and Boards/cs_debug/cs_debug_v1.sch (EAGLE design)
At the start: 168 parts, among them J1 J-JTAG-CORTEX_SMD, J19 Solar, J2 J-JTAG-CORTEX_SMD, J3 J-JTAG-CORTEX-NEEDLE6-LEGS, J4 J-SERIAL-PORT, J401 J-USB-HIROSE-MICRO-USB, J403 J-WURTH-USBC, Q10 2N7002P, Q3 FDN340P, Q4 2N7002P, Q5 FDN340P, Q6 2N7002P, Q7 FDN340P, Q8 2N7002P, Q9 FDN340P, U1 AP2120N-3.3TRG1, U10 OPA357AIDBVTG4, U11 DAC7574IDGS, U12 MCP73871T-2CCI/ML, U2 TLV1117LV33DCYR, U3 INA225AIDGK, U4 OPA357AIDBVTG4, U5 INA225AIDGK, U6 OPA357AIDBVTG4, U7 INA225AIDGK, U8 OPA357AIDBVTG4, U9 INA225AIDGK, Y101 32.768kHz, Y102 12mHz-12pF-K7

Commit message: Add USB connector and switch IC
Parts:
- removed C20: 10n, Capacitors:C-0402
- removed C21: 22u, Capacitors:C-0805
- removed C401: 2.2uF, Capacitors:C-0402
- removed C45: 2.2uF, Capacitors:C-0805
- removed J401: J-USB-HIROSE-MICRO-USB, Connectors:J-USB-HIROSE-MICRO-USB
- removed J403: J-WURTH-USBC, Connectors:J-WURTH-USBC
- removed R422, R423: 5.1k, Resistors:R-0603
- removed R7: 10k, Resistors:R-0402
- removed VR1, VR2, VR401, VR402, VR403: VARISTOR, Diodes:VARISTOR
- added C46: 2.2uF, Capacitors:C-0805
- added C47: 1u, Capacitors:C-0402
- added C48, C49, C50, C51, C52, C53: 0.1u, Capacitors:C-0402
- added C54: 4.7u, Capacitors:C-0402
- added C55, C56: 18pF, Capacitors:C-0402
- added J5: J-WURTH-USBC, Connectors:J-WURTH-USBC
- added JP14, JP15, JP16: JUMPER-SMT_2_NC_PASTE_NO-SILK, SparkFun-Jumpers:JUMPER-SMT_2_NC_PASTE_NO-SILK
- added L2: DLP11SN900HL2L, Inductors:DLP11SN900HL2L
- added R42, R43: 5.1k, Resistors:R-0603
- added R44, R45, R51, R52: 10k, Resistors:R-0402
- added R46, R47, R49, R50: 100k, Resistors:R-0402
- added R48: 12k, Resistors:R-0402
- added U$5: BGX50A, Diodes:BGX50A
- added U13: USB2412-DZK, Switches:USB2412-DZK
- added VR3, VR4: VARISTOR, Diodes:VARISTOR
- added Y1: HCM49-24.000MABJ-UT, Oscillators:HCM49-24.000MABJ-UT
- R204: MPN RC0402JR-07100KL -> ERJ-2GEJ104X; PART_NO RC0402JR-07100KL -> ERJ-2GEJ104X
Connections:
- removed net CC1: J403_CONNECTOR.CC1, R422.2
- removed net CC2: J403_CONNECTOR.CC2, R423.2
- removed net D+: J403_CONNECTOR.DP1, J403_CONNECTOR.DP2, VR1.1
- removed net D-: J403_CONNECTOR.DN1, J403_CONNECTOR.DN2, VR2.1
- removed net VBUS: C20.1, C21.1, C401.1, C45.1, D1.C, J401.VBUS, J403_CONNECTOR.VBUS, J403_CONNECTOR.VBUS1, J403_CONNECTOR.VBUS2, J403_CONNECTOR.VBUS3, L1.1, R7.2, U_INSTR_PROC.VBUS
- new net CC3: J5_CONNECTOR.CC1, R42.2
- new net CC4: J5_CONNECTOR.CC2, R43.2
- new net N$12: U13.TEST, U13.TEST1
- new net N$14: R45.1, U13.PRTPWR1
- new net N$15: D1.C, JP14.1
- new net N$16: R44.1, U13.PRTPWR2
- new net N$17: R48.2, U13.RBIAS
- new net N$18: R46.2, R47.1, U13.VBUS_DET
- new net N$19: C48.1, R49.1, U13.RESET_N
- new net N$20: C55.1, U13.XTALIN/CLKIN, Y1.1
- new net N$21: C56.1, U13.XTALOUT, Y1.2
- new net N$22: R50.2, U13.HS_IND
- new net N$23: R52.1, U13.NON_REMI
- new net N$24: R51.1, U13.SUSP_IND/NON_REM0
- new net USB_CONN_D_N: J5_CONNECTOR.DP1, J5_CONNECTOR.DP2, L2.3, U$5.AC1, VR3.1
- new net USB_CONN_D_P: J5_CONNECTOR.DN1, J5_CONNECTOR.DN2, L2.2, U$5.AC2, VR4.1
- new net USB_D_N: L2.4, U13.USBDM_UP
- new net USB_D_P: L2.1, U13.USBDP_UP
- new net USB_VBUS: C46.1, C47.1, J5_CONNECTOR.VBUS, J5_CONNECTOR.VBUS1, J5_CONNECTOR.VBUS2, J5_CONNECTOR.VBUS3, JP14.2, JP15.1, JP15.2, L1.1, R47.2, U$5.+, U_INSTR_PROC.VBUS
- net 3V3_INSTR_PROC: now also C49.1, C50.1, C51.1, C52.1, C53.1, C54.1, R44.2, R45.2, R49.2, R51.2, R52.2, U13.VDD33, U13.VDD33_2, U13.VDD33_3, U13.VDD33_4, U13.VDD33_5
- net DGND: now also C46.2, C47.2, C48.2, C49.2, C50.2, C51.2, C52.2, C53.2, C54.2, C55.2, C56.2, J5_CONNECTOR.GND, J5_CONNECTOR.GND1, J5_CONNECTOR.GND2, J5_CONNECTOR.GND3, J5_SHIELD.SHIELD, R42.1, R43.1, R46.1, R48.1, R50.1, U$5.-, U13.EPAD, VR3.2, VR4.2; no longer C20.2, C21.2, C401.2, J401.GND, J401.SHIELD, R7.1, VR401.2, VR402.2, VR403.2
- net GND: no longer C45.2, J403_CONNECTOR.GND, J403_CONNECTOR.GND1, J403_CONNECTOR.GND2, J403_CONNECTOR.GND3, J403_SHIELD.SHIELD, R422.1, R423.1, VR1.2, VR2.2
- net INSTR_PROC_USB_D_N: now also U13.USBDM_DN2; no longer J401.D-, VR403.1
- net INSTR_PROC_USB_D_P: now also U13.USBDP_DN2; no longer J401.D+, VR402.1
- net INSTR_PROC_USB_UOTGID: no longer J401.USBID, VR401.1
- net MAIN_USART_TX: now also JP16.2
- net MAIN_USB_DATA_N: now also U13.USBDM_DN1
- net MAIN_USB_DATA_P: now also U13.USBDP_DN1
- net UCTX_DBGRX: now also J5_CONNECTOR.SBU1, J5_CONNECTOR.SBU2, JP16.1; no longer J403_CONNECTOR.SBU1, J403_CONNECTOR.SBU2
Other:
- note added: "Add DLP11SN900SL2 and BGX50A"
- note added: "Battery Charger"
- note added: "Connection questionable"
- note added: "ESD protection"
- note added: "Extra Power Source (Solar)"
- note added: "USB Hub/Switch"
- note added: "USB Type-C Connector"
- note added: "pull-up for power pins; hub should not shutdown other devices"
- note removed: "Charger"
- note removed: "Power Sources and USB"
- note removed: "Switch to USB type-c and include a hub IC to provide power, data lines to each"
- moved on the sheet: C1, C18, C2, C205, C208, C3, D1, F2, J1, J19, JP10, JP11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
