File: debug/Schematics and Boards/cs_debug/cs_debug_v1.sch (EAGLE design)
At the start: 186 parts, among them J1 J-JTAG-CORTEX_SMD, J19 Solar, J2 J-JTAG-CORTEX_SMD, J3 J-JTAG-CORTEX-NEEDLE6-LEGS, J4 J-SERIAL-PORT, J5 J-WURTH-USBC, Q10 2N7002P, Q3 FDN340P, Q4 2N7002P, Q5 FDN340P, Q6 2N7002P, Q7 FDN340P, Q8 2N7002P, Q9 FDN340P, U1 AP2120N-3.3TRG1, U10 OPA357AIDBVTG4, U11 DAC7574IDGS, U12 MCP73871T-2CCI/ML, U13 USB2412-DZK, U2 TLV1117LV33DCYR, U3 INA225AIDGK, U4 OPA357AIDBVTG4, U5 INA225AIDGK, U6 OPA357AIDBVTG4, U7 INA225AIDGK, U8 OPA357AIDBVTG4, U9 INA225AIDGK, Y1 HCM49-24.000MABJ-UT, Y101 32.768kHz, Y102 12mHz-12pF-K7

Commit message: Add and name test points for debug board
Parts:
- removed C4: 68p, Capacitors:C-0402
- removed C5, C6: 0.1u, Capacitors:C-0402
- removed R10, R12, R14: 10k, Resistors:R-0402
- removed R11: 100k, Resistors:R-0402
- removed R13, R9: 249k, Resistors:R-0402
- removed R15: 5.1, Resistors:R-0603
- removed U3: INA225AIDGK, Amplifiers:INA225AIDGK
- removed U4: OPA357AIDBVTG4, Amplifiers:OPA357AIDBVTG4
- added C20: 680pF, Capacitors:C-0402
- added C21, C45: 0.1u, Capacitors:C-0402
- added R53, R55, R57: 10k, Resistors:R-0402
- added R54: 100k, Resistors:R-0402
- added R56: 249k, Resistors:R-0402
- added R58, R59: 5.1, Resistors:R-0603
- added TP_3V3_IPROC, TP_3V3_MEAS, TP_M_D_DA_VO, TP_M_D_OA_EN, TP_M_D_OA_N, TP_M_D_OA_P, TP_M_D_OA_VO, TP_M_D_SDN, TP_M_D_VN, TP_M_D_VOI, TP_M_P_DA_VO, TP_M_P_OA_N, TP_M_P_OA_P, TP_M_P_OA_VO, TP_M_P_SDN, TP_M_P_VN, TP_M_P_VOI, TP_M_S_DA_VO, TP_M_S_OA_EN, TP_M_S_OA_N, TP_M_S_OA_P, TP_M_S_OA_VO, TP_M_S_SDN, TP_M_S_VN, TP_M_S_VOI, TP_M_T_DA_VO, TP_M_T_OA_EN, TP_M_T_OA_N, TP_M_T_OA_P, TP_M_T_OA_VO, TP_M_T_SDN, TP_M_T_VN, TP_M_T_VOI, TP_SCL, TP_SDA, T_M_P_OA_EN: TPTP10SQ, TestPoints:TPTP10SQ
- added U14: INA225AIDGK, Amplifiers:INA225AIDGK
- added U15: OPA357AIDBVTG4, Amplifiers:OPA357AIDBVTG4
- C10, C13, C7: value 68p -> 680pF; MPN C0402C689D8GAC7867 -> C0402C681K8RAC7867; PART_NO C0402C689D8GAC7867 -> C0402C681K8RAC7867
- C11, C12, C14, C15, C8, C9: MPN C0402C104K8RACTU -> (none)
- R16, R24, R40: value 5.1 -> 249k; device Resistors:R-0603 -> Resistors:R-0402; MPN ERJ-3BQF5R1V -> ERA-2AEB2491X; PART_NO ERJ-3BQF5R1V -> ERA-2AEB2491X; TOL 1% -> 0,1%
- R17, R33: value 249k -> 10k; MPN ERA-2AEB2491X -> ERA-2AEB103X; PART_NO ERA-2AEB2491X -> ERA-2AEB103X; SPICEPREFIX (none) -> R; TOL 0,1% -> 0.1%
- R18, R34: value 10k -> 100k; MPN ERA-2AEB103X -> ERJ-2RKF1003X; PART_NO ERA-2AEB103X -> ERJ-2RKF1003X; SPICEPREFIX R -> (none); TOL 0.1% -> 1%
- R19, R35: value 100k -> 10k; MPN ERJ-2RKF1003X -> ERA-2AEB103X; PART_NO ERJ-2RKF1003X -> ERA-2AEB103X; TOL 1% -> 0.1%
- R20, R36: value 10k -> 249k; MPN ERA-2AEB103X -> ERA-2AEB2491X; PART_NO ERA-2AEB103X -> ERA-2AEB2491X
- R21, R37: value 249k -> 10k; MPN ERA-2AEB2491X -> ERJ-2RKF1002X; PART_NO ERA-2AEB2491X -> ERJ-2RKF1002X; TOL 0.1% -> 1%
- R22, R38: value 10k -> 5.1; device Resistors:R-0402 -> Resistors:R-0603; MPN ERJ-2RKF1002X -> ERJ-3BQF5R1V; PART_NO ERJ-2RKF1002X -> ERJ-3BQF5R1V
- renumbered JP11 to JP_VREG_SEL
Connections:
- net CM_DTR_DIFFAMP_N3 renamed CM_DIFFAMP_N3
- net CM_DTR_DIFFAMP_P3 renamed CM_DIFFAMP_P3
- removed net CM_DTR_OPAMP_ENABLE3: Q7.G, Q8.DRAIN, R27.1, U8.ENABLE
- removed net CM_DTR_OPAMP_N3: R28.1, R29.2, U8.IN-
- removed net CM_DTR_OPAMP_OUT3: Q7.S, R28.2, R31.1, U8.OUT
- removed net CM_DTR_OPAMP_P3: R25.2, R26.2, U8.IN+
- removed net CM_PROC_DIFFAMP_N1: C4.1, R15.2, U3.IN-
- removed net CM_PROC_DIFFAMP_P1: C4.2, R16.2, U3.IN+
- removed net CM_PROC_OPAMP_ENABLE1: Q3.G, Q4.DRAIN, R11.1, U4.ENABLE
- removed net CM_PROC_OPAMP_N1: R12.1, R13.2, U4.IN-
- removed net CM_PROC_OPAMP_OUT1: Q3.S, R12.2, R15.1, U4.OUT
- removed net CM_STORAGE_DIFFAMP_N1: C7.1, R23.2, U5.IN-
- removed net CM_STORAGE_DIFFAMP_P1: C7.2, R24.2, U5.IN+
- removed net CM_STORAGE_OPAMP_ENABLE1: Q5.G, Q6.DRAIN, R19.1, U6.ENABLE
- removed net CM_STORAGE_OPAMP_N1: R20.1, R21.2, U6.IN-
- removed net CM_STORAGE_OPAMP_OUT1: Q5.S, R20.2, R23.1, U6.OUT
- removed net CM_STORAGE_OPAMP_P1: R17.2, R18.2, U6.IN+
- removed net CM_TEMP_DIFFAMP_N1: C13.1, R39.2, U9.IN-
- removed net CM_TEMP_DIFFAMP_P1: C13.2, R40.2, U9.IN+
- removed net CM_TEMP_OPAMP_ENABLE1: Q10.DRAIN, Q9.G, R35.1, U10.ENABLE
- removed net CM_TEMP_OPAMP_N1: R36.1, R37.2, U10.IN-
- removed net CM_TEMP_OPAMP_OUT1: Q9.S, R36.2, R39.1, U10.OUT
- removed net CM_TEMP_OPAMP_P1: R33.2, R34.2, U10.IN+
- removed net CM__PROCOPAMP_P1: R10.2, R9.2, U4.IN+
- new net CM_DIFFAMP_N1: C20.1, R58.2, U14.IN-
- new net CM_DIFFAMP_N2: C13.1, R38.2, U9.IN-
- new net CM_DIFFAMP_N4: C7.1, R22.2, U5.IN-
- new net CM_DIFFAMP_P1: C20.2, R59.2, U14.IN+
- new net CM_DIFFAMP_P2: C13.2, R39.2, U9.IN+
- new net CM_DIFFAMP_P4: C7.2, R23.2, U5.IN+
- new net CM_OPAMP_ENABLE1: Q10.DRAIN, Q9.G, R54.1, TP_M_T_OA_EN.TP, U15.ENABLE
- new net CM_OPAMP_ENABLE2: Q5.G, Q6.DRAIN, R34.1, TP_M_S_OA_EN.TP, U10.ENABLE
- new net CM_OPAMP_ENABLE3: Q7.G, Q8.DRAIN, R27.1, TP_M_D_OA_EN.TP, U8.ENABLE
- new net CM_OPAMP_ENABLE4: Q3.G, Q4.DRAIN, R18.1, T_M_P_OA_EN.TP, U6.ENABLE
- new net CM_OPAMP_N1: R55.1, R56.2, TP_M_T_OA_N.TP, U15.IN-
- new net CM_OPAMP_N2: R35.1, R36.2, TP_M_S_OA_N.TP, U10.IN-
- new net CM_OPAMP_N3: R28.1, R29.2, TP_M_D_OA_N.TP, U8.IN-
- new net CM_OPAMP_N4: R19.1, R20.2, TP_M_P_OA_N.TP, U6.IN-
- new net CM_OPAMP_OUT1: Q9.S, R55.2, R58.1, TP_M_T_OA_VO.TP, U15.OUT
- new net CM_OPAMP_OUT2: Q5.S, R35.2, R38.1, TP_M_S_OA_VO.TP, U10.OUT
- new net CM_OPAMP_OUT3: Q7.S, R28.2, R31.1, TP_M_D_OA_VO.TP, U8.OUT
- new net CM_OPAMP_OUT4: Q3.S, R19.2, R22.1, TP_M_P_OA_VO.TP, U6.OUT
- new net CM_OPAMP_P1: R40.2, R53.2, TP_M_T_OA_P.TP, U15.IN+
- new net CM_OPAMP_P2: R24.2, R33.2, TP_M_S_OA_P.TP, U10.IN+
- new net CM_OPAMP_P3: R25.2, R26.2, TP_M_D_OA_P.TP, U8.IN+
- new net CM_OPAMP_P4: R16.2, R17.2, TP_M_P_OA_P.TP, U6.IN+
- net 3V3_INSTR_MEAS: now also C21.1, C45.1, R18.2, R21.2, R34.2, R37.2, R54.2, R57.2, TP_3V3_MEAS.TP, U14.V+, U15.V+; no longer C5.1, C6.1, R11.2, R14.2, R19.2, R22.2, R35.2, R38.2, U3.V+, U4.V+
- net 3V3_INSTR_PROC: now also TP_3V3_IPROC.TP
- net AGND: now also C21.2, C45.2, R20.1, R36.1, R56.1, U14.REF, U14.V-, U15.V-; no longer C5.2, C6.2, R13.1, R21.1, R37.1, U3.REF, U3.V-, U4.V-
- net CM_DTR_DCBIAS_SHUTDOWN: now also TP_M_D_SDN.TP
- net CM_DTR_DIFFAMP_OUT: now also TP_M_D_DA_VO.TP
- net CM_DTR_V_OFFSET_IN: now also TP_M_D_VOI.TP
- net CM_DTR_V_SENSE_N: now also TP_M_D_VN.TP
- net CM_PROC_DCBIAS_SHUTDOWN: now also R21.1, TP_M_P_SDN.TP; no longer R14.1
- net CM_PROC_DIFFAMP_GAIN0: now also U5.GS0; no longer U3.GS0
- net CM_PROC_DIFFAMP_GAIN1: now also U5.GS1; no longer U3.GS1
- net CM_PROC_DIFFAMP_OUT: now also TP_M_P_DA_VO.TP, U5.OUT; no longer U3.OUT
- net CM_PROC_V_OFFSET_IN: now also R16.1, TP_M_P_VOI.TP; no longer R9.1
- net CM_PROC_V_SENSE_N: now also R17.1, TP_M_P_VN.TP; no longer R10.1
- net CM_PROC_V_SENSE_P: now also R23.1; no longer R16.1
- net CM_STORAGE_DCBIAS_SHUTDOWN: now also R37.1, TP_M_S_SDN.TP; no longer R22.1
- net CM_STORAGE_DIFFAMP_GAIN0: now also U9.GS0; no longer U5.GS0
- net CM_STORAGE_DIFFAMP_GAIN1: now also U9.GS1; no longer U5.GS1
- net CM_STORAGE_DIFFAMP_OUT: now also TP_M_S_DA_VO.TP, U9.OUT; no longer U5.OUT
- net CM_STORAGE_V_OFFSET_IN: now also R24.1, TP_M_S_VOI.TP; no longer R17.1
- net CM_STORAGE_V_SENSE_N: now also R33.1, TP_M_S_VN.TP; no longer R18.1
- net CM_STORAGE_V_SENSE_P: now also R39.1; no longer R24.1
- net CM_TEMP_DCBIAS_SHUTDOWN: now also R57.1, TP_M_T_SDN.TP; no longer R38.1
- net CM_TEMP_DIFFAMP_GAIN0: now also U14.GS0; no longer U9.GS0
- net CM_TEMP_DIFFAMP_GAIN1: now also U14.GS1; no longer U9.GS1
- net CM_TEMP_DIFFAMP_OUT: now also TP_M_T_DA_VO.TP, U14.OUT; no longer U9.OUT
- net CM_TEMP_V_OFFSET_IN: now also R40.1, TP_M_T_VOI.TP; no longer R33.1
- net CM_TEMP_V_SENSE_N: now also R53.1, TP_M_T_VN.TP; no longer R34.1
- net CM_TEMP_V_SENSE_P: now also R59.1; no longer R40.1
- net INSTR_PROC_I2C_SCL: now also TP_SCL.TP
- net INSTR_PROC_I2C_SDA: now also TP_SDA.TP
Other:
- note added: "Daughter Board High-Side Current Monitor"
- note added: "Processor High-Side Current Monitor"
- note added: "Storage High-Side Current Monitor"
- note added: "Temp High-Side Current Monitor"
- note removed: "10x cap for larger RC constant"
- note removed: "A pun on temporary and temperature It is probably unnecessary to dedicate an entire channel to the temperature sensor, whose current draw is near negligible Instead, we may change this channel to be used for something else, most likely another signal from the daughter card"
- note removed: "Channel 0"
- note removed: "Channel 1"
- note removed: "Channel 2"
- note removed: "Channel 3"
- note removed: "May need to use a larger resistor (2512) because there are plenty of analog signals There are >=9 analog signals 1 for vense+ 4 for sense- 4 for DAC outputs"
- moved on the sheet: C10, C11, C12, C13, C14, C15, C7, C8, C9, JP1, JP2, JP3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

Commit message: Add backup micro-usb ports
Parts:
- removed JP14: JUMPER-SMT_2_NC_PASTE_NO-SILK, SparkFun-Jumpers:JUMPER-SMT_2_NC_PASTE_NO-SILK
- removed JP_VREG_SEL: JUMPER-SMT_3_1-NC_PASTE_NO-SILK, Connectors:JUMPER-SMT_3_1-NC_PASTE_NO-SILK
- removed TP_SDA: TPTP10SQ, TestPoints:TPTP10SQ
- added JP.USB.DDN, JP.USB.DDP, JP.USB.MDN, JP.USB.MDP, JP.VREG.SEL: JUMPER-SMT_3_1-NC_PASTE_NO-SILK, Connectors:JUMPER-SMT_3_1-NC_PASTE_NO-SILK
- added JP.USBM.DBG, JP.USBM.MAIN: JUMPER-SMT_2_NO_PASTEFREE, Connectors:JUMPER-SMT_2_NO_PASTEFREE
- added JP.VEXT: JUMPER-SMT_2_NC_PASTE_NO-SILK, SparkFun-Jumpers:JUMPER-SMT_2_NC_PASTE_NO-SILK
- added J_USB_DBG, J_USB_MAIN: USBABSMTDIP, ZX62D-AB-5P8:USBABSMTDIP
- added SDA: TPTP10SQ, TestPoints:TPTP10SQ
- added VR1, VR2, VR5, VR6, VR7, VR8: VARISTOR, Diodes:VARISTOR
- C46: device Capacitors:C-0805 -> Capacitors:C-0603; MPN (none) -> C0603C225K8RACTU; PART_NO (none) -> C0603C225K8RACTU
- L2: MPN (none) -> DLP11SN900HL2L; PART_NO (none) -> DLP11SN900HL2L
- R42, R43: MPN (none) -> ERJ-2GEJ512X; PART_NO (none) -> ERJ-2GEJ512X
- VR3, VR4: PART_NO (none) -> CG0603MLC-05E
- renumbered JP1 to JP.P.PROC, JP101 to JP.IP.AREF, JP102 to JP.IP.VDDIO, JP103 to JP.IP.ANA, JP104 to JP.IP.UTMI, JP105 to JP.IP.OUT, JP106 to JP.IP.CORE, JP107 to JP.IP.PLL, JP12 to JP.IP.RST, JP13 to JP.UART.VCC, JP15 to JP.USBC.VBUS, JP16 to JP.USB.USART, JP2 to JP.P.STOR, JP3 to JP.P.TEMP, JP4 to JP.P.DTR, JP5 to JP.EN.VMEAS, JP6 to JP.EN.VPROC, JP7 to JP.VDD.MAIN, JP8 to JP.UART.TX.IP, JP9 to JP.UART.RX.IP, TP_M_D_DA_VO to M.D.DA.VO, TP_M_D_OA_EN to M.D.OA.EN, TP_M_D_OA_N to M.D.OA.N, TP_M_D_OA_P to M.D.OA.P, TP_M_D_OA_VO to M.D.OA.VO, TP_M_D_SDN to M.D.SDN, TP_M_D_VN to M.D.VN, TP_M_D_VOI to M.D.VOI, TP_M_P_DA_VO to M.P.DA.VO, TP_M_P_OA_N to M.P.OA.N, TP_M_P_OA_P to M.P.OA.P, TP_M_P_OA_VO to M.P.OA.VO, TP_M_P_SDN to M.P.SDN, TP_M_P_VN to M.P.VN, TP_M_P_VOI to M.P.VOI, TP_M_S_DA_VO to M.S.DA.VO, TP_M_S_OA_EN to M.S.OA.EN, TP_M_S_OA_N to M.S.OA.N, TP_M_S_OA_P to M.S.OA.P, TP_M_S_OA_VO to M.S.OA.VO, TP_M_S_SDN to M.S.SDN, TP_M_S_VN to M.S.VN, TP_M_S_VOI to M.S.VOI, TP_M_T_DA_VO to M.T.DA.VO, TP_M_T_OA_EN to M.T.OA.EN, TP_M_T_OA_N to M.T.OA.N, TP_M_T_OA_P to M.T.OA.P, TP_M_T_OA_VO to M.T.OA.VO, TP_M_T_SDN to M.T.SDN, TP_M_T_VN to M.T.VN, TP_M_T_VOI to M.T.VOI, TP_SCL to SCL, T_M_P_OA_EN to M.P.OA.EN, U$5 to D2
Connections:
- new net HUB_INSTR_PROC_USB_D_N: JP.USB.DDN.3, U13.USBDM_DN2
- new net HUB_INSTR_PROC_USB_D_P: JP.USB.DDP.3, U13.USBDP_DN2
- new net HUB_MAIN_USB_DATA_N: U13.USBDM_DN1
- new net HUB_MAIN_USB_DATA_P: JP.USB.MDN.3, JP.USB.MDP.3, U13.USBDP_DN1
- new net USB_BKUP_DBG_D_N: JP.USB.DDN.1, J_USB_DBG.D-, VR5.1
- new net USB_BKUP_DBG_D_P: JP.USB.DDP.1, J_USB_DBG.D+, VR2.1
- new net USB_BKUP_DBG_OTGID: J_USB_DBG.USBID, VR1.1
- new net USB_BKUP_DBG_VBUS: JP.USBM.DBG.2, J_USB_DBG.VBUS
- new net USB_BKUP_MAIN_D_N: JP.USB.MDP.1, J_USB_MAIN.D-, VR8.1
- new net USB_BKUP_MAIN_D_P: JP.USB.MDN.1, J_USB_MAIN.D+, VR7.1
- new net USB_BKUP_MAIN_OTGID: J_USB_MAIN.USBID, VR6.1
- new net USB_BKUP_MAIN_VBUS: JP.USBM.MAIN.2, J_USB_MAIN.VBUS
- net GND: now also J_USB_DBG.GND, J_USB_DBG.SHIELD, J_USB_MAIN.GND, J_USB_MAIN.SHIELD, VR1.2, VR2.2, VR5.2, VR6.2, VR7.2, VR8.2
- net INSTR_PROC_I2C_SDA: now also SDA.TP; no longer TP_SDA.TP
- net INSTR_PROC_USB_D_N: now also JP.USB.DDN.2; no longer U13.USBDM_DN2
- net INSTR_PROC_USB_D_P: now also JP.USB.DDP.2; no longer U13.USBDP_DN2
- net MAIN_USB_DATA_N: now also JP.USB.MDN.2; no longer U13.USBDM_DN1
- net MAIN_USB_DATA_P: now also JP.USB.MDP.2; no longer U13.USBDP_DN1
- net N$15: now also JP.VEXT.1; no longer JP14.1
- net USB_VBUS: now also JP.USBM.DBG.1, JP.USBM.MAIN.1, JP.VEXT.2; no longer JP14.2
- net VCHRG_OUT: now also JP.VREG.SEL.3; no longer JP_VREG_SEL.3
- net VREG_IN: now also JP.VREG.SEL.2; no longer JP_VREG_SEL.2
- net VSRC_RAW: now also JP.VREG.SEL.1; no longer JP_VREG_SEL.1
Other:
- note added: "Floating bc internal pull-ups"
- note added: "USB Micro Connectors (backup for hub)"
- moved on the sheet: D1, J19, L1, R1, R48, R51, R52, S201

Commit message: Dbg board: subsystem organization
Did relative placement for all subsystems (processor, regulator, usb- hub, etc.)

It is unlikely that all components on this board can fit into a small footprint due to the size and number of components. Some further squeezing and optimization can be done, but part of the board will need to be larger to expose vertically accessed ports (debug).
Parts:
- removed JP.VEXT, JP10: JUMPER-SMT_2_NC_PASTE_NO-SILK, SparkFun-Jumpers:JUMPER-SMT_2_NC_PASTE_NO-SILK
- added JP.CHRG.MAIN, JP.EXT.PWR, JP.UART.RX, JP.UART.TX: JUMPER-SMT_2_NC_PASTE_NO-SILK, Connectors:JUMPER-SMT_2_NC_PASTE_NO-SILK
- JP.EN.VMEAS, JP.EN.VPROC, JP.P.DTR, JP.P.PROC, JP.P.STOR, JP.P.TEMP, JP.USB.USART, JP.USBC.VBUS, JP.VDD.MAIN: device SparkFun-Jumpers:JUMPER-SMT_2_NC_PASTE_NO-SILK -> Connectors:JUMPER-SMT_2_NC_PASTE_NO-SILK
- Y1: value HCM49-24.000MABJ-UT -> EPSON_TSX-3225_24.0000MF10Z-C3; device Oscillators:HCM49-24.000MABJ-UT -> Oscillators:EPSON_TSX-3225_24.0000MF10Z-C3; MPN (none) -> TSX-3225 24.0000MF10Z-C3; PART_NO (none) -> TSX-3225 24.0000MF10Z-C3
- renumbered S1 to S.NRST, S102 to S.ERASE, TP_3V3_IPROC to 3V3.IPROC, TP_3V3_MEAS to 3V3.MEAS
Connections:
- removed net GND: C18.2, C208.2, J19.1, J_USB_DBG.GND, J_USB_DBG.SHIELD, J_USB_MAIN.GND, J_USB_MAIN.SHIELD, S.NRST.1, VR1.2, VR2.2, VR5.2, VR6.2, VR7.2, VR8.2
- removed net N$12: U13.TEST, U13.TEST1
- new net N$7: J4.RX-I, JP.UART.TX.2
- new net N$9: J4.TX-O, JP.UART.RX.2
- new net VSRC: JP.EXT.PWR.2, JP.USBC.VBUS.2, JP.USBM.DBG.1, JP.USBM.MAIN.1, L1.1
- net DGND: now also C18.2, C208.2, J19.1, J_USB_DBG.GND, J_USB_DBG.SHIELD, J_USB_MAIN.GND, J_USB_MAIN.SHIELD, S.NRST.1, U13.TEST, U13.TEST1, VR1.2, VR2.2, VR5.2, VR6.2, VR7.2, VR8.2, Y1.1_GND, Y1.2_GND
- net HUB_MAIN_USB_DATA_N: now also JP.USB.MDN.3
- net HUB_MAIN_USB_DATA_P: no longer JP.USB.MDN.3
- net MAIN_USART_RX: now also JP.UART.RX.1; no longer J4.TX-O
- net MAIN_USART_TX: now also JP.UART.TX.1; no longer J4.RX-I
- net N$15: now also JP.EXT.PWR.1; no longer JP.VEXT.1
- net N$21: now also Y1.3; no longer Y1.2
- net USB_VBUS: no longer JP.USBC.VBUS.2, JP.USBM.DBG.1, JP.USBM.MAIN.1, JP.VEXT.2, L1.1
- net VCHRG_BATT: now also JP.CHRG.MAIN.1; no longer JP10.1
- net V_BATT_MAIN: now also JP.CHRG.MAIN.2; no longer JP10.2
Other:
- moved on the sheet: C55, C56

Commit message: Relative subsystem placement
still off board
Parts:
- added JP.USB.VBUSP: JUMPER-SMT_3_1-NC_PASTE_NO-SILK, Connectors:JUMPER-SMT_3_1-NC_PASTE_NO-SILK
Connections:
- removed net USB_VBUS: C46.1, C47.1, D2.+, J5_CONNECTOR.VBUS, J5_CONNECTOR.VBUS1, J5_CONNECTOR.VBUS2, J5_CONNECTOR.VBUS3, JP.USBC.VBUS.1, R47.2, U_INSTR_PROC.VBUS
- new net USBC_VBUS: C46.1, C47.1, D2.+, J5_CONNECTOR.VBUS, J5_CONNECTOR.VBUS1, J5_CONNECTOR.VBUS2, J5_CONNECTOR.VBUS3, JP.USB.VBUSP.3, JP.USBC.VBUS.1, R47.2
- new net USB_VBUS_IPROC: JP.USB.VBUSP.2, U_INSTR_PROC.VBUS
- net USB_BKUP_DBG_VBUS: now also JP.USB.VBUSP.1
Other:
- moved on the sheet: JP.USB.DDN, JP.USB.DDP, JP.USB.MDN, JP.USB.MDP

Commit message: DBG-Manual checks & minor cleanup
Parts:
- added JP.HUB.VDD: JUMPER-SMT_2_NC_PASTE_NO-SILK, Connectors:JUMPER-SMT_2_NC_PASTE_NO-SILK
- added R7: 1M, Resistors:R-0402
- renumbered J_DEBUG_TO_MAIN_HEADER to J_DBG_TO_MAIN_HDR
Connections:
- net N$17 renamed USB_RBIAS
- net N$18 renamed HUB_USB_VBUS
- net N$19 renamed USB_HUB_RST
- net N$22 renamed USB_HS_IND
- net N$23 renamed USB_NONRMV1
- net N$24 renamed USB_NONRMV0
- removed net N$20: C55.1, U13.XTALIN/CLKIN, Y1.1
- removed net N$21: C56.1, U13.XTALOUT, Y1.3
- new net USB_HUB_VDD: JP.HUB.VDD.2, U13.VDD33, U13.VDD33_2, U13.VDD33_3, U13.VDD33_4, U13.VDD33_5
- new net USB_XIN: C55.1, R7.2, U13.XTALIN/CLKIN, Y1.1
- new net USB_XOUT: C56.1, R7.1, U13.XTALOUT, Y1.3
- net 3V3_INSTR_PROC: now also JP.HUB.VDD.1; no longer U13.VDD33, U13.VDD33_2, U13.VDD33_3, U13.VDD33_4, U13.VDD33_5

Commit message: BOM cleanup and initial CAM
Parts:
- C11, C12, C14, C15, C21, C45, C8, C9: MPN (none) -> C0402C104K8RACTU
- J1, J2: PART_NO (none) -> FTSH-105-01-L-DV-K-TR
- J4: PART_NO (none) -> PH1-06-UA
- J5: PART_NO (none) -> 632723100011
- J_USB_DBG: MPN (none) -> ZX62D-AB-5P8(30); PART_NO (none) -> ZX62D-AB-5P8(30)
- J_USB_MAIN: MPN (none) -> ZX62D-AB-5P8(30); PAR_NO (none) -> ZX62D-AB-5P8(30)
- R1: MPN (none) -> ERJ-S1D0R00U; PART_NO (none) -> ERJ-S1D0R00U
