File: debug/Schematics and Boards/cs_debug/cs_debug_v1.sch (EAGLE design)
At the start: 241 parts, among them J1 J-JTAG-CORTEX_SMD, J19 Solar, J2 J-JTAG-CORTEX_SMD, J3 J-JTAG-CORTEX-NEEDLE6-LEGS, J4 J-SERIAL-PORT, J5 J-WURTH-USBC, Q10 2N7002P, Q3 FDN340P, Q4 2N7002P, Q5 FDN340P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

Commit message: Minor changes and notes
Nothing fundamental changed here; mostly preparation for a round of revisions
Parts:
- C10, C13, C20, C7: value 680pF -> 270nF; device Capacitors:C-0402 -> Capacitors:C-0603; MPN C0402C681K8RAC7867 -> C0603C274K8PACTU; PART_NO C0402C681K8RAC7867 -> C0603C274K8PACTU; TC C0G -> X5R
- C208: device Capacitors:C-0402 -> Capacitors:C-0603
- R42, R43: MPN ERJ-2GEJ512X -> ERJ-3EKF5101V; PART_NO ERJ-2GEJ512X -> ERJ-3EKF5101V
Other:
- note added: "BKUP FOR MAIN IS SWAPPED!!"
Changed lines of the file:
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@@
 <attribute name="PART_NO" value="ERJ-2GEJ274X"/>
 </part>
-<part name="C208" library="Capacitors" deviceset="C-" device="0402" value="4.7u">
+<part name="C208" library="Capacitors" deviceset="C-" device="0603" value="4.7u">
 <attribute name="MPN" value="C0603C475M8PACTU"/>
 <attribute name="PART_NO" value="C0603C475M8PACTU"/>
@@
 <part name="GND20" library="Supplies" deviceset="GND" device=""/>
 <part name="R42" library="Resistors" deviceset="R-" device="0603" value="5.1k">
-<attribute name="MPN" value="ERJ-2GEJ512X"/>
-<attribute name="PART_NO" value="ERJ-2GEJ512X"/>
+<attribute name="MPN" value="ERJ-3EKF5101V"/>
+<attribute name="PART_NO" value="ERJ-3EKF5101V"/>
 </part>
 <part name="R43" library="Resistors" deviceset="R-" device="0603" value="5.1k">
-<attribute name="MPN" value="ERJ-2GEJ512X"/>
-<attribute name="PART_NO" value="ERJ-2GEJ512X"/>
+<attribute name="MPN" value="ERJ-3EKF5101V"/>
+<attribute name="PART_NO" value="ERJ-3EKF5101V"/>
 </part>
 <part name="FRAME3" library="frames" library_urn="urn:adsk.eagle:library:229" deviceset="FRAME_C_L" device=""/>
@@
 <attribute name="TOL" value="1%"/>
 </part>
-<part name="C20" library="Capacitors" deviceset="C-" device="0402" value="680pF">
-<attribute name="MPN" value="C0402C681K8RAC7867 "/>
-<attribute name="PART_NO" value="C0402C681K8RAC7867 "/>
-<attribute name="TC" value="C0G"/>
+<part name="C20" library="Capacitors" deviceset="C-" device="0603" value="270nF">
+<attribute name="MPN" value="C0603C274K8PACTU"/>
+<attribute name="PART_NO" value="C0603C274K8PACTU"/>
+<attribute name="TC" value="X5R"/>
 <attribute name="TOL" value="0.5pF"/>
 <attribute name="VOLTAGE" value="10V"/>
@@
 <attribute name="TOL" value="1%"/>
 </part>
-<part name="C13" library="Capacitors" deviceset="C-" device="0402" value="680pF">
-<attribute name="MPN" value="C0402C681K8RAC7867 "/>
-<attribute name="PART_NO" value="C0402C681K8RAC7867 "/>
-<attribute name="TC" value="C0G"/>
+<part name="C13" library="Capacitors" deviceset="C-" device="0603" value="270nF">
+<attribute name="MPN" value="C0603C274K8PACTU"/>
+<attribute name="PART_NO" value="C0603C274K8PACTU"/>
+<attribute name="TC" value="X5R"/>
 <attribute name="TOL" value="0.5pF"/>
 <attribute name="VOLTAGE" value="10V"/>
@@
 <attribute name="TOL" value="1%"/>
 </part>
-<part name="C10" library="Capacitors" deviceset="C-" device="0402" value="680pF">
-<attribute name="MPN" value="C0402C681K8RAC7867 "/>
-<attribute name="PART_NO" value="C0402C681K8RAC7867 "/>
-<attribute name="TC" value="C0G"/>
+<part name="C10" library="Capacitors" deviceset="C-" device="0603" value="270nF">
+<attribute name="MPN" value="C0603C274K8PACTU"/>
+<attribute name="PART_NO" value="C0603C274K8PACTU"/>
+<attribute name="TC" value="X5R"/>
 <attribute name="TOL" value="0.5pF"/>
 <attribute name="VOLTAGE" value="10V"/>
@@
 <attribute name="TOL" value="1%"/>
 </part>
-<part name="C7" library="Capacitors" deviceset="C-" device="0402" value="680pF">
-<attribute name="MPN" value="C0402C681K8RAC7867 "/>
-<attribute name="PART_NO" value="C0402C681K8RAC7867 "/>
-<attribute name="TC" value="C0G"/>
+<part name="C7" library="Capacitors" deviceset="C-" device="0603" value="270nF">
+<attribute name="MPN" value="C0603C274K8PACTU"/>
+<attribute name="PART_NO" value="C0603C274K8PACTU"/>
+<attribute name="TC" value="X5R"/>
 <attribute name="TOL" value="0.5pF"/>
 <attribute name="VOLTAGE" value="10V"/>
@@
 <wire x1="124.46" y1="360.68" x2="25.4" y2="360.68" width="0.381" layer="97" style="longdash"/>
 <wire x1="149.86" y1="360.68" x2="132.08" y2="360.68" width="0.381" layer="97" style="longdash"/>
+<text x="342.9" y="327.66" size="1.778" layer="91">BKUP FOR MAIN IS SWAPPED!!</text>
 </plain>
 <instances>
