File: daughter/Schematics and Boards/CSv2_exp_board/CSv2_exp_board.brd (EAGLE design)
At the start: 38.1 x 44.5 mm, 144 parts, among them J1 HIROSE-DF40_44-PIN_CONNECTORS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, J2 J-SERIAL-PORT, J3 CORTEX_DEBUG_SMD, J4 SJ-43514-SMT, J5 HIROSE-DF40_44-PIN_CONNECTORS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, J6 ATTINY_AVR_DEBUG, J7 J-USB-HIROSE-MICRO-USB, SW1 SPST_TACT-KMR2, SW2 SPST_TACT-KMR2, T1 TPTP10SQ, T10 TPTP10SQ, T11 TPTP10SQ, T2 TPTP10SQ, T3 TPTP10SQ, T4 TPTP10SQ, T5 TPTP10SQ, T6 TPTP10SQ, T7 TPTP10SQ, T8 TPTP10SQ, T9 TPTP10SQ, U1 LOADSWITCH-MIC94164, U10 LOADSWITCH-MIC94164, U11 BMI160, U12 TLV320DAC26IRHB, U13 ADG839YKSZ-500RL7KS_6_ADI-L, U14 LOADSWITCH-MIC94164, U15 LP2980AIM5-2.5/NOPBMF05A_TEX-L, U16 NCP553SQ18T1GSC-82AB_ONS-L, U17 ATTINY817-MFRQFN24_RX4MC-L_AT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, U18 MPL3115A2, U19 ATSAMD21G18_QFN, U2 ADA4841-1YRJZ-R7RJ_6-L, U3 Value, U4 RFM69HCW, U5 Value, U6 Value, U7 LOADSWITCH-MIC94164, U8 LOADSWITCH-MIC94164, U9 LOADSWITCH-MIC94164, X1 32.768kHz, X2 32.768kHz, X3 uFL, X4 uFL, X5 uFL, X6 uFL

Commit message: DTR-v1.1 after moving LoRa to the top
Parts:
- moved J3 24.0 mm to (37.0, 11.6)
- moved T10 21.6 mm to (36.8, 18.5)
- moved T9 20.3 mm to (33.0, 18.5)
- moved T11 18.9 mm to (34.9, 18.5)
- moved JP11 18.5 mm to (32.6, 9.91), turned to 90 degrees
- moved C11 16.9 mm to (32.5, 14.0), turned to 180 degrees
- moved U1 16.8 mm to (32.5, 12.9), turned to 270 degrees
- moved C10 16.8 mm to (32.4, 11.8), turned to 180 degrees
- moved JP2 16.7 mm to (32.5, 15.8)
- moved X4 14.9 mm to (48.3, 20.1)
- moved A1 13.8 mm to (49.0, 10.0)
- moved C3 13.8 mm to (50.1, 4.15)
- moved C5 13.8 mm to (46.1, 5.54)
- moved C9 13.0 mm to (37.8, 30.7), flipped to the bottom
- moved R28 12.3 mm to (45.3, 15.3), turned to 240 degrees
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Connections:
- net +3V3_RFM_PWR: now also U6.9; no longer U6.3
- net +3V3_SAMD_PWR: now also U6.3; no longer U6.9
- net MEAS_RFM: now also U6.8; no longer U6.4
- net MEAS_SAMD: now also U6.4; no longer U6.8
Routing:
- net SAMD_!RESET: track 21.6 -> 46.6 mm, vias 3 -> 2
- net MEAS_SAMD: track 17.6 -> 40.0 mm
- net BUS1_SERCOM_P0: track 60.5 -> 39.1 mm
- net +3V3_NMEAS: track 35.2 -> 51.0 mm
- net MEAS_RFM: track 20.7 -> 34.4 mm, vias 2 -> 1
- net EN_RADIO: track 25.0 -> 37.4 mm, vias 3 -> 2
- net +3V3_RFM: track 4.46 -> 15.9 mm
- net +3V3_SAMD: track 21.9 -> 30.6 mm, vias 3 -> 4
- net SWCLK: track 13.1 -> 21.9 mm
- net GND: track 48.1 -> 40.1 mm, vias 73 -> 30
- net D_P: track 14.7 -> 7.47 mm
- net SWDIO: track 13.5 -> 20.5 mm
- net D_N: track 14.1 -> 7.42 mm
- net BUS1_SERCOM_P1: track 44.6 -> 38.0 mm
- net BUS1_GPIO1: track 36.0 -> 29.4 mm
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Other:
- board size 38.1 x 44.5 mm -> 50.8 x 44.5 mm
- board text added: "AT RESET"
- board text added: "CommonSense Daughter Board v1 Eve Hu 7/2/2020"
- board text added: "SAMD DEBUG"
- board text removed: "A RESET"
- board text removed: "CommonSense Daughter Board v1 Eve Hu 06/29/2020"
- board text removed: "SDEBUG"

Commit message: DTR-rounded inner corners, adjusted silkscreen texts, added CAM/gerber
Parts:
- J4: value SJ-43514-SMT -> SJ-43514-SMTC; device CommonSense-DTR-v1:CUI_SJ-43514-SMT -> CommonSense-DTR-v1:CUI_SJ-43514-SMT-TEMP
- U4: device Radios:RFM-MOD -> CommonSense-DTR-v1:RFM-MOD
- moved SW1 1.20 mm to (10.4, 32.2)
- moved J2 0.67 mm to (13.1, 43.0)
- moved X3 0.63 mm to (1.45, 36.2)
- moved R7 0.52 mm to (3.07, 33.6)
- moved J7 0.43 mm to (26.7, 42.7)
- moved ASCL 0.33 mm to (33.8, 6.81)
- moved ASDA 0.33 mm to (33.8, 5.49)
- moved JP16 0.25 mm to (32.3, 3.66)
- moved JP3 0.23 mm to (15.3, 24.0)
- moved X6 0.23 mm to (4.55, 31.9)
- moved JP8 0.23 mm to (17.9, 24.0)
- turned C21 to 180 degrees
- renumbered D_IN to DIN, D_OUT to DOUT
Routing:
- net N$12: track 7.69 -> 5.77 mm
- net MEAS_SAMD: track 40.0 -> 41.1 mm
- net +3V3_IMU_IN: track 4.27 -> 3.46 mm
- net GND: vias 30 -> 50
Other:
- outline, holes or cut-outs redrawn
