File: debug/Schematics and Boards/cs_debug_v1/cs_debug_v1.brd (EAGLE design)
At the start: 83.3 x 62.2 mm, 241 parts, among them J1 J-JTAG-CORTEX_SMD, J19 Solar, J2 J-JTAG-CORTEX_SMD, J3 J-JTAG-CORTEX-NEEDLE6-LEGS, J4 J-SERIAL-PORT, J5 J-WURTH-USBC, Q10 2N7002P, Q3 FDN340P, Q4 2N7002P, Q5 FDN340P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

Commit message: DBG: Fix DFM issues for 7PCB
Parts:
- J.USB.DBG, J.USB.MN: value USBABSMTDIP -> J-USB-HIROSE-MICRO-USB; device ZX62D-AB-5P8:ZX62D-AB-5P8 -> Connectors:USB-THRU-ZX62D-AB-5P8
