File: daughter/Schematics and Boards/CSv2_exp_board_v2/CSv2.1_exp_board.sch (EAGLE design)
At the start: 103 parts, among them J1 HIROSE-DF40_50-PIN_CONNECTORS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, J3 CORTEX_DEBUG_SMD, J4 SJ-43514-SMTC, J6 ATTINY_AVR_DEBUG, J7 J-USB-HIROSE-MICRO-USB, SW1 SPST_TACT-KMR2, SW2 SPST_TACT-KMR2, U1 LOADSWITCH-MIC94164, U10 LOADSWITCH-MIC94164, U11 BMI160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

Commit message: DTR - fixed BOM
Parts:
- added C33: 0.1u, Capacitors:C-0402
- added LED2: (no value), Diodes:LEDCHIPLED_0603
- added R12: 1k, Resistors:R-0402
- C27, C28, C31, C35, C36: DESC (none) -> CAP CER 0.1UF 10V X7R 0402; MPN (none) -> CC0402KRX7R6BB104; PARTNO (none) -> CC0402KRX7R6BB104
- C32: DESC (none) -> CAP CER 1UF 10V X7S 0402; MANUFACTURER (none) -> TDK; MPN (none) -> C1005X7S1A105K050BC; PARTNO (none) -> C1005X7S1A105K050BC
- J1: MANUFACTURER (none) -> Hirose; MPN (none) -> DF40C-50DP-0.4V(51); PARTNO (none) -> DF40C-50DP-0.4V(51)
- JP16: BOM (none) -> EXCLUDE
- LED1: DESC (none) -> LED RED CLEAR CHIP SMD; MANUFACTURER (none) -> Kingbright; MPN (none) -> APT1608SURCK; PARTNO (none) -> APT1608SURCK; TYPE (none) -> LED
- R11: value (none) -> 1k; DESC (none) -> Thick Film Resistors - SMD 0402 1Kohms 1% AEC-Q200; MPN (none) -> ERJ-2RKF1001X; PARTNO (none) -> ERJ-2RKF1001X; TOL (none) -> 1%; TYPE (none) -> Resistor
- R2: DESC RES SMD 82.5KOHM 0.1% 1/16W 0402 -> RES SMD 100K OHM 0.1% 1/16W 0402; HEIGHT 0.4mm -> 0.35mm; MANUFACTURER (none) -> Yageo; MPN ERA-2AEB8252X -> RT0402BRD07100KL; PARTNO ERA-2AEB8252X -> RT0402BRD07100KL
- R30: value 1.2n -> 0R; DESC FIXED IND 1.2NH 390MA 100 MOHM -> RES 0 OHM JUMPER 1/16W 0402; MANUFACTURER Murata -> Stackpole; MPN LQP15MN1N2W02D -> RMCF0402ZT0R00; PARTNO LQP15MN1N2W02D -> RMCF0402ZT0R00; TOL 0.05nH -> Jumper; TYPE Inductor -> Resistor
- R8: value (none) -> 0R; MPN (none) -> RMCF0402ZT0R00; PARTNO (none) -> RMCF0402ZT0R00; TYPE (none) -> Resistor
- U$1: MPN (none) -> SGTL5000XNLA3R2; PARTNO (none) -> SGTL5000XNLA3R2
- renumbered L1 to R30
Connections:
- net IN+ renamed N$3
- new net DTR_DETECT_LED: LED2.A, R12.2
- net +1V8_CODEC: now also C33.1
- net DTR_DETECT: now also R12.1
- net GND: now also C33.2, LED2.C

Commit message: DTR-fixed silk screem and switched to a new pressure sensor
Parts:
- removed C40: 10u, Capacitors:C-0603
- removed C47, C48: 0.1u, Capacitors:C-0402
- removed U18: MPL3115A2, Sensors:MPL3115A2
- added U206: MS5637, Sensors:MS5637
- C26, R27, R28, R30: BOM (none) -> EXCLUDE
- renumbered LED1 to RED_LED, LED2 to GREEN_LED
Connections:
- removed net N$10: C48.1, U18.CAP
- net +3V3_BARO: now also U206.VDD; no longer C40.2, C47.1, U18.V, U18.VIO
- net DTR_BUS2_GPIO0: no longer U18.INT1
- net DTR_BUS2_P0/I2C_SDA: now also U206.SDA; no longer U18.SDA
- net DTR_BUS2_P1/I2C_SCL: now also U206.SCL; no longer U18.SCL
- net GND: now also U206.GND; no longer C40.1, C47.2, C48.2, U18.GND
Other:
- note removed: "I2C 7-BIT Address: 0x60 8-bit READ: 0xC1 8-bit WRITE: 0xC0"

Commit message: DTR - added notes to the schematic
Other:
- note added: "I2C 7-BIT Address: 1110110b (0x76)"
- note added: "I2C ADDR: 0001010b (0x0A)"
- note added: "PRESSURE SENSOR-MS5637"
- note removed: "PRESSURE SENSOR-MPL3115"
Changed lines of the file:
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@@
 <wire x1="233.68" y1="127" x2="233.68" y2="2.54" width="0.1524" layer="94" style="shortdash"/>
 <wire x1="154.94" y1="127" x2="396.24" y2="127" width="0.1524" layer="94" style="shortdash"/>
-<text x="254" y="76.2" size="2.54" layer="94">PRESSURE SENSOR-MPL3115</text>
+<text x="254" y="76.2" size="2.54" layer="94">PRESSURE SENSOR-MS5637</text>
 <wire x1="154.94" y1="127" x2="2.54" y2="127" width="0.1524" layer="94" style="shortdash"/>
 <wire x1="154.94" y1="200.66" x2="2.54" y2="200.66" width="0.1524" layer="94" style="shortdash"/>
@@
 SDO-&gt;VDDIO: 0x69
 F_MAX=1000kHz</text>
+<text x="271.78" y="27.94" size="1.778" layer="97" rot="MR0">I2C 7-BIT Address:
+1110110b (0x76)
+</text>
 </plain>
 <instances>
@@
 <text x="180.34" y="261.62" size="2.54" layer="94">ATTINY PWR</text>
 <wire x1="236.22" y1="271.78" x2="236.22" y2="2.54" width="0.1524" layer="94" style="shortdash"/>
+<text x="78.74" y="17.78" size="1.778" layer="97">I2C ADDR: 0001010b (0x0A)</text>
 </plain>
 <instances>

Commit message: DTR: update SGTL5000 library part according to the SDFM
Parts:
- U4: device CommonSense-DTR-v1:RFM95C -> Radios:RFM95C
Changed lines of the file:
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@@
 </part>
 <part name="+3V5" library="Supplies" deviceset="+3V3" device=""/>
-<part name="U4" library="CommonSense-DTR-v1" deviceset="RFM95" device="C" value="RFM69HCW">
+<part name="U4" library="Radios" deviceset="RFM95" device="C" value="RFM69HCW">
 <attribute name="DESC" value="RX TXRX MODULE ISM &lt; 1GHZ SMD"/>
 <attribute name="MPN" value="RFM95CW"/>
