File: main/Schematics and Boards/CSv2.1/cs_v2.1.sch (EAGLE design)
At the start: 78 parts, among them J101 J-JTAG-CORTEX-NEEDLE6-LEGS, J301 HIROSE-DF40_50-PIN_CONNECTORS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, J302 HIROSE-DF40_50-PIN_CONNECTORS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, Q1 DMG3415UFY4Q-7F, U1 NCP708MU330TAG, U101 ATSAMD51, U2 W25N01GVZEIG, U201 COULOMB-MAX17262, U202 MAX77827BEWC+T, U203 SENSOR-SI7006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

Commit message: Rename 'base' to 'main' for consistency in terminology
Parts:
- Q1: MP DMG3415U-7 -> DMG3415UFY4Q-7; MPN DMG3415U-7 -> DMG3415UFY4Q-7; PART_NO DMG3415U-7 -> DMG3415UFY4Q-7
- R207: device Resistors:R-0603 -> Resistors:R-0402; MANUFACTURER (none) -> Ohmite; MPN ERJ-2BQFR24X -> KDV06DR240ET; PART_NO ERJ-2BQFR24X -> KDV06DR240ET
Other:
- note added: "Address 0x36"
- note added: "Address 0x40"
Changed lines of the file:
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@@
 <attribute name="TOL" value="0.1%"/>
 </part>
-<part name="R207" library="Resistors" deviceset="R-" device="0603" value="0.24">
-<attribute name="MPN" value="ERJ-2BQFR24X"/>
-<attribute name="PART_NO" value="ERJ-2BQFR24X"/>
+<part name="R207" library="Resistors" deviceset="R-" device="0402" value="0.24">
+<attribute name="MANUFACTURER" value="Ohmite"/>
+<attribute name="MPN" value="KDV06DR240ET"/>
+<attribute name="PART_NO" value="KDV06DR240ET"/>
 <attribute name="TOL" value="0.5%"/>
 </part>
@@
 <part name="GND16" library="Supplies" deviceset="GND" device=""/>
 <part name="Q1" library="Switches" deviceset="DMG3415UFY4Q-7" device="F">
-<attribute name="MP" value="DMG3415U-7"/>
-<attribute name="MPN" value="DMG3415U-7"/>
-<attribute name="PART_NO" value="DMG3415U-7"/>
+<attribute name="MP" value="DMG3415UFY4Q-7"/>
+<attribute name="MPN" value="DMG3415UFY4Q-7"/>
+<attribute name="PART_NO" value="DMG3415UFY4Q-7"/>
 </part>
 <part name="R3" library="Resistors" deviceset="R-" device="0402" value="100k">
@@
 <wire x1="121.92" y1="71.12" x2="121.92" y2="15.24" width="0.1524" layer="91"/>
 <wire x1="121.92" y1="15.24" x2="119.38" y2="12.7" width="0.1524" layer="91"/>
+<label x="121.92" y="30.48" size="1.778" layer="95" rot="R90"/>
 </segment>
 </net>
@@
 <wire x1="124.46" y1="71.12" x2="124.46" y2="15.24" width="0.1524" layer="91"/>
 <wire x1="124.46" y1="15.24" x2="121.92" y2="12.7" width="0.1524" layer="91"/>
+<label x="124.46" y="30.48" size="1.778" layer="95" rot="R90"/>
 </segment>
 </net>
@@
 <wire x1="127" y1="71.12" x2="127" y2="15.24" width="0.1524" layer="91"/>
 <wire x1="127" y1="15.24" x2="124.46" y2="12.7" width="0.1524" layer="91"/>
+<label x="127" y="30.48" size="1.778" layer="95" rot="R90"/>
 </segment>
 </net>
@@
 <wire x1="129.54" y1="71.12" x2="129.54" y2="15.24" width="0.1524" layer="91"/>
 <wire x1="129.54" y1="15.24" x2="127" y2="12.7" width="0.1524" layer="91"/>
+<label x="129.54" y="30.48" size="1.778" layer="95" rot="R90"/>
 </segment>
 </net>
@@
 Estimate typical 260 mΩ for total 0.5Ω
 to account for ~200mA of current</text>
+<text x="258.318" y="35.56" size="1.778" layer="97">Address 0x40</text>
+<text x="111.76" y="147.32" size="1.778" layer="97">Address 0x36</text>
 </plain>
 <instances>
